Commit message: Got p3dx and p3at urdfs in order.  Renamed "center" wheel to caster.

File: description/urdf/pioneer3dx_body.xacro (robot description, xacro)
@@ -6,5 +6,5 @@
 	   xmlns:xacro="http://ros.org/wiki/xacro"
 	   >
-	<include filename="$(find p2os_urdf)/defs/pioneer3dx_wheel.xacro"/>
+	<xacro:include filename="$(find amr_robots_description)/urdf/pioneer3dx_wheel.xacro"/>
 	<!-- Chassis description -->
 	<link name="base_link">
@@ -21,5 +21,5 @@
 			<origin xyz="-0.045 0 0.148" rpy="0 0 0"/>
 			<geometry name="pioneer_geom">
-				<mesh filename="package://p2os_urdf/meshes/p3dx_meshes/chassis.stl"/>
+				<mesh filename="package://amr_robots_description/meshes/p3dx_meshes/chassis.stl"/>
 			</geometry>
 			<material name="ChassisRed">
@@ -30,5 +30,5 @@
 			<origin xyz="-0.045 0 0.148" rpy="0 0 0"/>
 				<geometry>
-					<mesh filename="package://p2os_urdf/meshes/p3at_meshes/chassis.stl"/>
+					<mesh filename="package://amr_robots_description/meshes/p3at_meshes/chassis.stl"/>
 				</geometry>
 		</collision>
@@ -48,5 +48,5 @@
 			<origin xyz="0 0 0" rpy="0 0 0"/>
 			<geometry name="pioneer_geom">
-				<mesh filename="package://p2os_urdf/meshes/p3dx_meshes/top.stl"/>
+				<mesh filename="package://amr_robots_description/meshes/p3dx_meshes/top.stl"/>
 			</geometry>
 			<material name="TopBlack">
@@ -82,5 +82,5 @@
 		<origin xyz="0 0 0" rpy="0 0 0"/>
 		<geometry name="pioneer_geom">
-			<mesh filename="package://p2os_urdf/meshes/p3dx_meshes/swivel.stl"/>
+			<mesh filename="package://amr_robots_description/meshes/p3dx_meshes/swivel.stl"/>
 		</geometry>
 		<material name="swivel">
@@ -109,5 +109,5 @@
 		<origin xyz="0 0 0" rpy="0 0 0"/>
 		<geometry name="pioneer_geom">
-			<mesh filename="package://p2os_urdf/meshes/p3dx_meshes/center_hubcap.stl"/>
+			<mesh filename="package://amr_robots_description/meshes/p3dx_meshes/center_hubcap.stl"/>
 		</geometry>
 		<material name="swivel">
@@ -144,5 +144,5 @@
 		<origin xyz="0 0 0" rpy="0 0 0"/>
 		<geometry name="pioneer_geom">
-			<mesh filename="package://p2os_urdf/meshes/p3dx_meshes/center_wheel.stl"/>
+			<mesh filename="package://amr_robots_description/meshes/p3dx_meshes/center_wheel.stl"/>
 		</geometry>
 		<material name="WheelBlack">
@@ -153,5 +153,5 @@
 		<origin xyz="0 0 0" rpy="${-3.1415927/2.0} 0 0"/>
 		<geometry>
-			<!--<mesh filename="package://p2os_urdf/meshes/p3dx_meshes/center_wheel.stl"/>-->
+			<!--<mesh filename="package://amr_robots_description/meshes/p3dx_meshes/center_wheel.stl"/>-->
 			<cylinder radius="0.0375" length="0.01"/>
 		</geometry>
@@ -170,5 +170,5 @@
 			<origin xyz="0 0 0" rpy="0 0 0"/>
 			<geometry>
-				<mesh filename="package://p2os_urdf/meshes/p3dx_meshes/left_hubcap.stl"/>
+				<mesh filename="package://amr_robots_description/meshes/p3dx_meshes/left_hubcap.stl"/>
 			</geometry>
 			<material name="HubcapYellow">
@@ -179,5 +179,5 @@
 			<origin xyz="0 0 0" rpy="${-3.1415927/2.0} 0 0"/>
 			<geometry>
-				<!--<mesh filename="package://p2os_urdf/meshes/p3dx_meshes/center_wheel.stl"/>-->
+				<!--<mesh filename="package://amr_robots_description/meshes/p3dx_meshes/center_wheel.stl"/>-->
 				<cylinder radius="0.09" length="0.01"/>
 			</geometry>
@@ -194,5 +194,5 @@
 			<origin xyz="0 0 0" rpy="0 0 0"/>
 			<geometry>
-				<mesh filename="package://p2os_urdf/meshes/p3dx_meshes/left_wheel.stl"/>
+				<mesh filename="package://amr_robots_description/meshes/p3dx_meshes/left_wheel.stl"/>
 			</geometry>
 			<material name="WheelBlack">
@@ -213,5 +213,5 @@
 			<origin xyz="0 0 0" rpy="0 0 0"/>
 			<geometry>
-				<mesh filename="package://p2os_urdf/meshes/p3dx_meshes/right_hubcap.stl"/>
+				<mesh filename="package://amr_robots_description/meshes/p3dx_meshes/right_hubcap.stl"/>
 			</geometry>
 			<material name="HubcapYellow">
@@ -222,5 +222,5 @@
 		<origin xyz="0 0 0" rpy="${-3.1415927/2.0} 0 0"/>
 		<geometry>
-			<!--<mesh filename="package://p2os_urdf/meshes/p3dx_meshes/center_wheel.stl"/>-->
+			<!--<mesh filename="package://amr_robots_description/meshes/p3dx_meshes/center_wheel.stl"/>-->
 			<cylinder radius="0.09" length="0.01"/>
 		</geometry>
@@ -240,5 +240,5 @@
 			<origin xyz="0 0 0" rpy="0 0 0"/>
 			<geometry>
-				<mesh filename="package://p2os_urdf/meshes/p3dx_meshes/right_wheel.stl"/>
+				<mesh filename="package://amr_robots_description/meshes/p3dx_meshes/right_wheel.stl"/>
 			</geometry>
 			<material name="WheelBlack">
@@ -266,5 +266,5 @@
 			<origin xyz="0 0 0" rpy="0 0 0"/>
 			<geometry name="pioneer_geom">
-				<mesh filename="package://p2os_urdf/meshes/p3dx_meshes/front_sonar.stl"/>
+				<mesh filename="package://amr_robots_description/meshes/p3dx_meshes/front_sonar.stl"/>
 			</geometry>
 			<material name="SonarYellow">
@@ -297,5 +297,5 @@
 			<origin xyz="0 0 0" rpy="0 0 0"/>
 			<geometry name="pioneer_geom">
-				<mesh filename="package://p2os_urdf/meshes/p3dx_meshes/back_sonar.stl"/>
+				<mesh filename="package://amr_robots_description/meshes/p3dx_meshes/back_sonar.stl"/>
 			</geometry>
 			<material name="SonarYellow">
