Commit message: renamed _wheel_link to just _wheel. Added Jaco2 arms to LX Devil.

File: description/urdf/pioneer-lx-devil.urdf.xacro (robot description, xacro)
@@ -1,4 +1,4 @@
 <?xml version="1.0"?>
-<robot name="pioneer-lx-devil" xmlns:xacro="http://ros.org/wiki/xacro">
+<robot name="pioneer-lx-devil" xmlns:xacro="http://www.ros.org/wiki/xacro">
   <!-- TODO share pioneer lx mobile robot components with pioneer-lx urdf -->
   <link name="base_link">
@@ -22,17 +22,17 @@
   </link>
   <!-- right wheel -->
-  <link name="r_wheel_link">
+  <link name="r_wheel">
     <inertial>
       <mass value="1.1" />   <!-- kg -->
       <inertia ixx="0.02" ixy="0" ixz="0" iyy="0.02" iyz="0" izz="0.01" />
     </inertial>
-    <visual name="r_wheel_link_dumb_visual">
-      <geometry name="r_wheel_link_dumb_visual_geom">
+    <visual name="r_wheel_dumb_visual">
+      <geometry name="r_wheel_dumb_visual_geom">
         <cylinder radius="0.100" length="0.05" />
       </geometry>
       <origin rpy="1.570796 0 0" />
     </visual>
-    <collision name="r_wheel_link_collision">
-      <geometry name="r_wheel_link_collision_geom">
+    <collision name="r_wheel_collision">
+      <geometry name="r_wheel_collision_geom">
         <cylinder radius="0.100" length="0.05" />
       </geometry>
@@ -41,17 +41,17 @@
   </link>
   <!-- left wheel -->
-  <link name="l_wheel_link">
+  <link name="l_wheel">
     <inertial>
       <mass value="1.1" />   <!-- kg -->
       <inertia ixx="0.02" ixy="0" ixz="0" iyy="0.02" iyz="0" izz="0.01" />
     </inertial>
-    <visual name="l_wheel_link_dumb_visual">
-      <geometry name="l_wheel_link_dumb_visual_geom">
+    <visual name="l_wheel_dumb_visual">
+      <geometry name="l_wheel_dumb_visual_geom">
         <cylinder radius="0.100" length="0.05" />
       </geometry>
       <origin rpy="1.570796 0 0" />
     </visual>
-    <collision name="l_wheel_link_collision">
-      <geometry name="l_wheel_link_collision_geom">
+    <collision name="l_wheel_collision">
+      <geometry name="l_wheel_collision_geom">
         <cylinder radius="0.100" length="0.05" />
       </geometry>
@@ -63,12 +63,28 @@
     <origin xyz="0 0.2 0.1" rpy="0 0 0" />
     <parent link="base_link" />
-    <child link="r_wheel_link" />
+    <child link="r_wheel" />
   </joint>
   <joint name="l_wheel_joint" type="continuous">
     <origin xyz="0 -0.2 0.1" rpy="0 0 0" />
     <parent link="base_link" />
-    <child link="l_wheel_link" />
+    <child link="l_wheel" />
   </joint>
   <!-- arms -->
-  <xacro:include filename="$(find kinova_description)/urdf/jaco2_arm.xacro />
+  <xacro:include filename="$(find kinova_description)/urdf/jaco2_arm.xacro" />
+  <link name="right_arm_mount">
+  </link>
+  <link name="left_arm_mount">
+  </link>
+  <xacro:jaco2_arm parent="right_arm_mount" prefix="right_" />
+  <xacro:jaco2_arm parent="left_arm_mount" prefix="left_" />
+  <joint name="right_arm_attach" type="fixed">
+    <child link="right_arm_mount" />
+    <parent link="base_link" />
+    <origin xyz="-0.020 0.184 1.240" rpy="0 0 0" />
+  </joint>
+  <joint name="left_arm_attach" type="fixed">
+    <child link="left_arm_mount" />
+    <parent link="base_link" />
+    <origin xyz="-0.020 -0.184 1.240" rpy="0 0 0" />
+  </joint>
 </robot>

File: description/urdf/pioneer-lx.urdf.xacro (robot description, xacro)
@@ -21,17 +21,17 @@
   </link>
   <!-- right wheel -->
-  <link name="r_wheel_link">
+  <link name="r_wheel">
     <inertial>
       <mass value="1.1" />   <!-- kg -->
       <inertia ixx="0.02" ixy="0" ixz="0" iyy="0.02" iyz="0" izz="0.01" />
     </inertial>
-    <visual name="r_wheel_link_dumb_visual">
-      <geometry name="r_wheel_link_dumb_visual_geom">
+    <visual name="r_wheel_dumb_visual">
+      <geometry name="r_wheel_dumb_visual_geom">
         <cylinder radius="0.100" length="0.05" />
       </geometry>
       <origin rpy="1.570796 0 0" />
     </visual>
-    <collision name="r_wheel_link_collision">
-      <geometry name="r_wheel_link_collision_geom">
+    <collision name="r_wheel_collision">
+      <geometry name="r_wheel_collision_geom">
         <cylinder radius="0.100" length="0.05" />
       </geometry>
@@ -40,17 +40,17 @@
   </link>
   <!-- left wheel -->
-  <link name="l_wheel_link">
+  <link name="l_wheel">
     <inertial>
       <mass value="1.1" />   <!-- kg -->
       <inertia ixx="0.02" ixy="0" ixz="0" iyy="0.02" iyz="0" izz="0.01" />
     </inertial>
-    <visual name="l_wheel_link_dumb_visual">
-      <geometry name="l_wheel_link_dumb_visual_geom">
+    <visual name="l_wheel_dumb_visual">
+      <geometry name="l_wheel_dumb_visual_geom">
         <cylinder radius="0.100" length="0.05" />
       </geometry>
       <origin rpy="1.570796 0 0" />
     </visual>
-    <collision name="l_wheel_link_collision">
-      <geometry name="l_wheel_link_collision_geom">
+    <collision name="l_wheel_collision">
+      <geometry name="l_wheel_collision_geom">
         <cylinder radius="0.100" length="0.05" />
       </geometry>
@@ -62,10 +62,10 @@
     <origin xyz="0 0.2 0.1" rpy="0 0 0" />
     <parent link="base_link" />
-    <child link="r_wheel_link" />
+    <child link="r_wheel" />
   </joint>
   <joint name="l_wheel_joint" type="continuous">
     <origin xyz="0 -0.2 0.1" rpy="0 0 0" />
     <parent link="base_link" />
-    <child link="l_wheel_link" />
+    <child link="l_wheel" />
   </joint>
 </robot>

Commit message: Added PTU and Kinect. Changed wheels to fixed for use with real robot (will need to be real joints for Gazebo's controller)

File: description/urdf/pioneer-lx-devil.urdf.xacro (robot description, xacro)
@@ -1,5 +1,7 @@
 <?xml version="1.0"?>
 <robot name="pioneer-lx-devil" xmlns:xacro="http://www.ros.org/wiki/xacro">
-  <!-- TODO share pioneer lx mobile robot components with pioneer-lx urdf -->
+  <!-- TODO share pioneer lx mobile robot components with pioneer-lx urdf by
+including macro. -->
+  <!-- TODO update Pioneer LX, deck and plinth with real meshes. -->
   <link name="base_link">
     <!-- base_link origin point is center of rotation, on the floor. -->
@@ -59,11 +61,11 @@
     </collision>
   </link>
-  <!-- wheel joints -->
-  <joint name="r_wheel_joint" type="continuous">
+  <!-- wheel joints. only used in gazebo, real robot velocity is controlled as a unit, not individual wheel motion. -->
+  <joint name="r_wheel_joint" type="fixed"> <!--  type="continuous" -->
     <origin xyz="0 0.2 0.1" rpy="0 0 0" />
     <parent link="base_link" />
     <child link="r_wheel" />
   </joint>
-  <joint name="l_wheel_joint" type="continuous">
+  <joint name="l_wheel_joint" type="fixed"> <!-- type="continuous" -->
     <origin xyz="0 -0.2 0.1" rpy="0 0 0" />
     <parent link="base_link" />
@@ -88,3 +90,50 @@
     <origin xyz="-0.020 -0.184 1.240" rpy="0 0 0" />
   </joint>
+  <!-- "plinth" plus deck (temporary model until we have meshes) -->
+  <link name="plinth">
+    <visual name="plinth_dumb_visual">
+      <geometry name="plinth_dumb_visual_geom">
+        <box size="0.18 0.2476 0.99" />
+        <!-- <origin xyz="-0.02 0 0.867" /> -->
+      </geometry>
+    </visual>
+    <collision name="plinth_dumb_collision">
+      <geometry name="plinth_dumb_collision_geom">
+        <box size="0.18 0.2476 0.99" />
+        <!-- <origin xyz="-0.02 0 0.867" /> -->
+      </geometry>
+    </collision>
+  </link>
+  <joint name="plinth_joint" type="fixed">
+    <parent link="base_link" />
+    <child link="plinth" />
+    <origin xyz="-0.02 0 0.867" />
+  </joint>
+ <!-- PTU -->
+  <xacro:include filename="$(find flir_ptu_description)/urdf/d46.urdf.xacro" />
+  <ptu_d46 name="ptu" />
+  <joint name="ptu_base_mount" type="fixed">
+    <parent link="plinth" />
+    <child link="ptu_base_link" />
+    <origin xyz="0 0 0.457" /> <!-- centered on top of plinth. TODO this is a temporary position. note mounting holes for PTU will actually offset a bit, check whether d46.urdf.xacro uses mounting hole, bottom, or center of ptu as its origin. -->
+  </joint>
+  <!-- kinect -->
+  <link name="kinect">
+    <visual name="kinect_visual">
+      <geometry name="kinect_visual_geom">
+        <box size="0.07 0.25 0.065" />
+        <origin xyz="0.03 0 0.035" />
+      </geometry>
+    </visual>
+    <collision name="kinect_collision">
+      <geometry name="kinect_visual_geom">
+        <box size="0.07 0.25 0.065" />
+        <origin xyz="0.03 0 0.035" />
+      </geometry>
+    </collision>
+  </link>
+  <joint name="kinect_mount" type="fixed">
+    <parent link="ptu_mount_link" />
+    <child  link="kinect" />
+  </joint>
 </robot>

Commit message: gave some things colors

File: description/urdf/pioneer-lx-devil.urdf.xacro (robot description, xacro)
@@ -15,4 +15,7 @@
       </geometry>
       <origin xyz="0 0 0.2" rpy="0 0 0" />
+      <material name="lx_red_mat">
+        <color rgba="0.8 0.1 0.1 1.0" />
+      </material>
     </visual>
     <collision name="base_link_dumb_collision">
@@ -34,4 +37,7 @@
       </geometry>
       <origin rpy="1.570796 0 0" />
+      <material name="lx_grey_mat">
+        <color rgba="0.8 0.8 0.8 1.0" />
+      </material>
     </visual>
     <collision name="r_wheel_collision">
@@ -53,4 +59,7 @@
       </geometry>
       <origin rpy="1.570796 0 0" />
+      <material name="lx_grey_mat">
+        <color rgba="0.8 0.8 0.8 1.0" />
+      </material>
     </visual>
     <collision name="l_wheel_collision">
@@ -97,4 +106,7 @@
         <!-- <origin xyz="-0.02 0 0.867" /> -->
       </geometry>
+      <material name="plinth_darkgrey_mat">
+        <color rgba="0.2 0.2 0.2 1.0" />
+      </material>
     </visual>
     <collision name="plinth_dumb_collision">
@@ -125,4 +137,7 @@
         <origin xyz="0.03 0 0.035" />
       </geometry>
+      <material name="kinect_black_mat">
+        <color rgba="0.0 0.0 0.0 1.0" />
+      </material>
     </visual>
     <collision name="kinect_collision">

Commit message: set arm mounting positions to new lower position

File: description/urdf/pioneer-lx-devil.urdf.xacro (robot description, xacro)
@@ -81,5 +81,5 @@
     <child link="l_wheel" />
   </joint>
-  <!-- Jaco2 arms.
+  <!-- Jaco2 arms, using lower upward-pointing mounting option.
        The kinova_description package is contained in the
        Kinovarobotics jaco_ros repository. As of 2/4/2015, you must
@@ -97,10 +97,10 @@
     <child link="right_arm_mount" />
     <parent link="base_link" />
-    <origin xyz="-0.020 0.184 1.240" rpy="0 0 0" />
+    <origin xyz="-0.020 0.184 1.1384" rpy="0 0 0" />
   </joint>
   <joint name="left_arm_attach" type="fixed">
     <child link="left_arm_mount" />
     <parent link="base_link" />
-    <origin xyz="-0.020 -0.184 1.240" rpy="0 0 0" />
+    <origin xyz="-0.020 -0.184 1.1384" rpy="0 0 0" />
   </joint>
   <!-- "plinth" plus deck (temporary model until we have meshes) -->

Commit message: Replace some squares with mesh references. fix syntax of p3at urdf

File: description/urdf/pioneer-lx-devil.urdf.xacro (robot description, xacro)
@@ -106,7 +106,8 @@
   <!-- "plinth" plus deck (temporary model until we have meshes) -->
   <link name="plinth">
-    <visual name="plinth_dumb_visual">
-      <geometry name="plinth_dumb_visual_geom">
-        <box size="0.18 0.2476 0.99" />
+    <visual name="plinth_visual">
+      <geometry name="plinth_visual_geom">
+        <mesh filename="package://amr_robots_description/meshes/pioneer-lx/plinth_hull.stl" />
+        <!-- box size="0.18 0.2476 0.99" / -->
         <!-- <origin xyz="-0.02 0 0.867" /> -->
       </geometry>
@@ -117,5 +118,6 @@
     <collision name="plinth_dumb_collision">
       <geometry name="plinth_dumb_collision_geom">
-        <box size="0.18 0.2476 0.99" />
+        <mesh filename="package://amr_robots_description/meshes/pioneer-lx/plinth_hull.stl" />
+        <!-- box size="0.18 0.2476 0.99" / -->
         <!-- <origin xyz="-0.02 0 0.867" /> -->
       </geometry>

File: description/urdf/pioneer-lx.urdf.xacro (robot description, xacro)
@@ -8,14 +8,16 @@
     </inertial>
     <visual name="base_link_dumb_visual">
-      <geometry name="base_link_dumb_visual_geom">
-        <box size="0.697 0.5 0.333" />
+      <geometry name="base_link_visual_geom">
+        <mesh filename="package://amr_robots_description/meshes/pioneer-lx/pioneer-lx_visual.stl" />
+        <!-- box size="0.697 0.5 0.333" / -->
       </geometry>
-      <origin xyz="0 0 0.2" rpy="0 0 0" />
+      <origin xyz="0 0 0.0" rpy="0 0 0" />
     </visual>
-    <collision name="base_link_dumb_collision">
-      <geometry name="base_link_dumb_collision_geom">
-        <box size="0.697 0.5 0.333" />
+    <collision name="base_link_collision">
+      <geometry name="base_link_collision_geom">
+        <mesh filename="package://amr_robots_description/meshes/pioneer-lx/pioneer-lx_hull.stl" />
+        <!-- box size="0.697 0.5 0.333" / -->
       </geometry>
-      <origin xyz="0 0 0.2" rpy="0 0 0" />
+      <origin xyz="0 0 0.0" rpy="0 0 0" />
     </collision>
   </link>
@@ -26,4 +28,6 @@
       <inertia ixx="0.02" ixy="0" ixz="0" iyy="0.02" iyz="0" izz="0.01" />
     </inertial>
+<!--
+TODO separate out pioner lx wheels in visual model
     <visual name="r_wheel_dumb_visual">
       <geometry name="r_wheel_dumb_visual_geom">
@@ -32,4 +36,5 @@
       <origin rpy="1.570796 0 0" />
     </visual>
+   -->
     <collision name="r_wheel_collision">
       <geometry name="r_wheel_collision_geom">
@@ -45,4 +50,5 @@
       <inertia ixx="0.02" ixy="0" ixz="0" iyy="0.02" iyz="0" izz="0.01" />
     </inertial>
+<!--
     <visual name="l_wheel_dumb_visual">
       <geometry name="l_wheel_dumb_visual_geom">
@@ -51,4 +57,5 @@
       <origin rpy="1.570796 0 0" />
     </visual>
+   -->
     <collision name="l_wheel_collision">
       <geometry name="l_wheel_collision_geom">

File: description/urdf/pioneer3at.urdf.xacro (robot description, xacro)
@@ -359,4 +359,5 @@
   </plugin>
 </gazebo>
+</xacro:macro>
 <xacro:p3at_front suffix="left" reflect="1"/>
 <xacro:p3at_front suffix="right" reflect="-1"/>

Commit message: Fixed positions of new meshes. added standin box for LX deck.

File: description/urdf/pioneer-lx-devil.urdf.xacro (robot description, xacro)
@@ -3,5 +3,4 @@
   <!-- TODO share pioneer lx mobile robot components with pioneer-lx urdf by
 including macro. -->
-  <!-- TODO update Pioneer LX, deck and plinth with real meshes. -->
   <link name="base_link">
     <!-- base_link origin point is center of rotation, on the floor. -->
@@ -10,18 +9,19 @@
       <inertia ixx="1" ixy="0" ixz="0" iyy="1" iyz="0" izz="1" />
     </inertial>
-    <visual name="base_link_dumb_visual">
-      <geometry name="base_link_dumb_visual_geom">
-        <box size="0.697 0.5 0.333" />
+    <visual name="base_link_visual">
+      <geometry name="base_link_visual_geom">
+        <mesh filename="package://amr_robots_description/meshes/pioneer-lx/pioneer-lx_visual.stl" scale="0.001 0.001 0.001" />
+        <!-- box size="0.697 0.5 0.333" / -->
       </geometry>
-      <origin xyz="0 0 0.2" rpy="0 0 0" />
+      <origin xyz="0 0 0" rpy="0 0 1.570796" />
       <material name="lx_red_mat">
         <color rgba="0.8 0.1 0.1 1.0" />
       </material>
     </visual>
-    <collision name="base_link_dumb_collision">
-      <geometry name="base_link_dumb_collision_geom">
-        <box size="0.697 0.5 0.333" />
+    <collision name="base_link_collision">
+      <geometry name="base_link_collision_geom">
+        <box size="0.697 0.5 0.35" />
       </geometry>
-      <origin xyz="0 0 0.2" rpy="0 0 0" />
+      <origin xyz="0 0 0.200" rpy="0 0 0" />
     </collision>
   </link>
@@ -32,4 +32,6 @@
       <inertia ixx="0.02" ixy="0" ixz="0" iyy="0.02" iyz="0" izz="0.01" />
     </inertial>
+<!--
+TODO separate out pioner lx wheels in visual model
     <visual name="r_wheel_dumb_visual">
       <geometry name="r_wheel_dumb_visual_geom">
@@ -41,4 +43,5 @@
       </material>
     </visual>
+-->
     <collision name="r_wheel_collision">
       <geometry name="r_wheel_collision_geom">
@@ -54,4 +57,5 @@
       <inertia ixx="0.02" ixy="0" ixz="0" iyy="0.02" iyz="0" izz="0.01" />
     </inertial>
+<!--
     <visual name="l_wheel_dumb_visual">
       <geometry name="l_wheel_dumb_visual_geom">
@@ -63,4 +67,5 @@
       </material>
     </visual>
+   -->
     <collision name="l_wheel_collision">
       <geometry name="l_wheel_collision_geom">
@@ -81,4 +86,49 @@
     <child link="l_wheel" />
   </joint>
+  <!-- pioneer lx deck -->
+  <link name="deck">
+    <visual name="deck_visual">
+      <geometry name="deck_visual_geom">
+        <box size="0.407 0.437 0.076" />
+      </geometry>
+      <material name="lx_deck_mat">
+        <color rgba="0 0 0 1" />
+      </material>
+    </visual>
+    <collision name="deck_collision">
+      <geometry name="deck_collision_geom">
+        <box size="0.407 0.437 0.076" />
+      </geometry>
+    </collision>
+  </link>
+  <joint name="deck_joint" type="fixed">
+    <origin xyz="0.075 0 0.410" rpy="0 0 0" />
+    <parent link="base_link" />
+    <child link="deck" />
+  </joint>
+  <!-- "plinth" -->
+  <link name="plinth">
+    <visual name="plinth_visual">
+      <geometry name="plinth_visual_geom">
+        <mesh filename="package://amr_robots_description/meshes/pioneer-lx/pioneer-lx-plinth.stl" scale="0.001 0.001 0.001" />
+        <!-- box size="0.18 0.2476 0.99" / -->
+      </geometry>
+      <material name="plinth_darkgrey_mat">
+        <color rgba="0.2 0.2 0.2 1.0" />
+      </material>
+    </visual>
+    <collision name="plinth_collision">
+      <geometry name="plinth_collision_geom">
+        <mesh filename="package://amr_robots_description/meshes/pioneer-lx/pioneer-lx-plinth.stl" scale="0.001 0.001 0.001" />
+        <!-- box size="0.18 0.2476 0.99" / -->
+        <origin xyz="-0.02 0 0.867" />
+      </geometry>
+    </collision>
+  </link>
+  <joint name="plinth_joint" type="fixed">
+    <parent link="base_link" />
+    <child link="plinth" />
+    <origin xyz="-0.11 0 0.448" />
+  </joint>
   <!-- Jaco2 arms, using lower upward-pointing mounting option.
        The kinova_description package is contained in the
@@ -88,47 +138,23 @@
    -->
   <xacro:include filename="$(find kinova_description)/urdf/jaco2_arm.xacro" />
+  <link name="left_arm_mount">
+  </link>
   <link name="right_arm_mount">
   </link>
-  <link name="left_arm_mount">
-  </link>
+  <xacro:jaco2_arm parent="left_arm_mount" prefix="left_" />
   <xacro:jaco2_arm parent="right_arm_mount" prefix="right_" />
-  <xacro:jaco2_arm parent="left_arm_mount" prefix="left_" />
+  <joint name="left_arm_attach" type="fixed">
+    <child link="left_arm_mount" />
+    <parent link="base_link" />
+    <origin xyz="-0.020 0.184 1.1384" rpy="0 0 0" />
+  </joint>
   <joint name="right_arm_attach" type="fixed">
     <child link="right_arm_mount" />
     <parent link="base_link" />
-    <origin xyz="-0.020 0.184 1.1384" rpy="0 0 0" />
-  </joint>
-  <joint name="left_arm_attach" type="fixed">
-    <child link="left_arm_mount" />
-    <parent link="base_link" />
     <origin xyz="-0.020 -0.184 1.1384" rpy="0 0 0" />
   </joint>
-  <!-- "plinth" plus deck (temporary model until we have meshes) -->
-  <link name="plinth">
-    <visual name="plinth_visual">
-      <geometry name="plinth_visual_geom">
-        <mesh filename="package://amr_robots_description/meshes/pioneer-lx/plinth_hull.stl" />
-        <!-- box size="0.18 0.2476 0.99" / -->
-        <!-- <origin xyz="-0.02 0 0.867" /> -->
-      </geometry>
-      <material name="plinth_darkgrey_mat">
-        <color rgba="0.2 0.2 0.2 1.0" />
-      </material>
-    </visual>
-    <collision name="plinth_dumb_collision">
-      <geometry name="plinth_dumb_collision_geom">
-        <mesh filename="package://amr_robots_description/meshes/pioneer-lx/plinth_hull.stl" />
-        <!-- box size="0.18 0.2476 0.99" / -->
-        <!-- <origin xyz="-0.02 0 0.867" /> -->
-      </geometry>
-    </collision>
-  </link>
-  <joint name="plinth_joint" type="fixed">
-    <parent link="base_link" />
-    <child link="plinth" />
-    <origin xyz="-0.02 0 0.867" />
-  </joint>
  <!-- PTU
-    The flir_ptu_description package is from the flir_ptu repository:
+    The flir_ptu_description package is either from system packages in
+    /opt/ros/... or from source repository
     https://github.com/ros-drivers/flir_ptu
   -->
@@ -138,5 +164,5 @@
     <parent link="plinth" />
     <child link="ptu_base_link" />
-    <origin xyz="0 0 0.457" /> <!-- centered on top of plinth. TODO this is a temporary position. note mounting holes for PTU will actually offset a bit, check whether d46.urdf.xacro uses mounting hole, bottom, or center of ptu as its origin. -->
+    <origin xyz="0.152 0.03 0.91" />
   </joint>
   <!-- kinect -->
@@ -161,4 +187,5 @@
     <parent link="ptu_mount_link" />
     <child  link="kinect" />
+    <origin xyz="0 0 0.0325" />
   </joint>
 </robot>

File: description/urdf/pioneer-lx.urdf.xacro (robot description, xacro)
@@ -7,17 +7,15 @@
       <inertia ixx="1" ixy="0" ixz="0" iyy="1" iyz="0" izz="1" />
     </inertial>
-    <visual name="base_link_dumb_visual">
+    <visual name="base_link_visual">
       <geometry name="base_link_visual_geom">
-        <mesh filename="package://amr_robots_description/meshes/pioneer-lx/pioneer-lx_visual.stl" />
-        <!-- box size="0.697 0.5 0.333" / -->
+        <mesh filename="package://amr_robots_description/meshes/pioneer-lx/pioneer-lx_visual.stl" scale="0.001 0.001 0.001" />
       </geometry>
-      <origin xyz="0 0 0.0" rpy="0 0 0" />
+      <origin xyz="0 0 0.0" rpy="0 0 1.570796" />
     </visual>
     <collision name="base_link_collision">
       <geometry name="base_link_collision_geom">
-        <mesh filename="package://amr_robots_description/meshes/pioneer-lx/pioneer-lx_hull.stl" />
-        <!-- box size="0.697 0.5 0.333" / -->
+        <box size="0.7 0.5 0.35" />
       </geometry>
-      <origin xyz="0 0 0.0" rpy="0 0 0" />
+      <origin xyz="0 0 0.2" rpy="0 0 0" />
     </collision>
   </link>
@@ -76,3 +74,24 @@
     <child link="l_wheel" />
   </joint>
+  <!-- pioneer lx deck -->
+  <link name="deck">
+    <visual name="deck_visual">
+      <geometry name="deck_visual_geom">
+        <box size="0.407 0.437 0.076" />
+      </geometry>
+      <material name="lx_deck_mat">
+        <color rgba="0 0 0 1" />
+      </material>
+    </visual>
+    <collision name="deck_collision">
+      <geometry name="deck_collision_geom">
+        <box size="0.407 0.437 0.076" />
+      </geometry>
+    </collision>
+  </link>
+  <joint name="deck_joint" type="fixed">
+    <origin xyz="0.075 0 0.410" rpy="0 0 0" />
+    <parent link="base_link" />
+    <child link="deck" />
+  </joint>
 </robot>
