Commit message: Fix launch files for good joint_state_publishers params. Added misc utility launch and rqt cconfiguration.

File: description/urdf/pioneer-lx-devil.urdf.xacro (robot description, xacro)
@@ -5,8 +5,4 @@
   <link name="base_link">
     <!-- base_link origin point is center of rotation, on the floor. -->
-    <inertial>
-      <mass value="57.8" /> <!-- 60 kg minus each wheel -->
-      <inertia ixx="1" ixy="0" ixz="0" iyy="1" iyz="0" izz="1" />
-    </inertial>
     <visual name="base_link_visual">
       <geometry name="base_link_visual_geom">
@@ -26,4 +22,15 @@
     </collision>
   </link>
+  <!-- for some reason KDL wants this to be a separate link -->
+  <link name="robot_mass">
+    <inertial>
+      <mass value="57.8" /> <!-- 60 kg minus each wheel -->
+      <inertia ixx="1" ixy="0" ixz="0" iyy="1" iyz="0" izz="1" />
+    </inertial>
+  </link>
+  <joint name="base_link_mass_attach">
+    <parent link="base_link">
+    <child link="base_link_mass">
+  </joint>
   <!-- right wheel -->
   <link name="r_wheel">

Commit message: separate inertial node for kdl

File: description/urdf/pioneer-lx-devil.urdf.xacro (robot description, xacro)
@@ -30,6 +30,6 @@
   </link>
   <joint name="base_link_mass_attach">
-    <parent link="base_link">
-    <child link="base_link_mass">
+    <parent link="base_link" />
+    <child link="base_link_mass" />
   </joint>
   <!-- right wheel -->
