Commit message: rotate arm mounting joints to face front, more testing tbd

File: description/urdf/pioneer-lx-devil.urdf (robot description, URDF)
Before this commit: robot pioneer-lx-devil, 37 links, 36 joints
Joints:
- joint left_arm_attach: origin xyz=-0.020 0.184 1.1384 rpy=0 0 0 -> xyz=-0.020 0.184 1.1384 rpy=0 0 1.5707
- joint right_arm_attach: origin xyz=-0.020 -0.184 1.1384 rpy=0 0 0 -> xyz=-0.020 -0.184 1.1384 rpy=0 0 1.5707

File: description/urdf/pioneer-lx-devil.urdf.xacro (robot description, xacro)
@@ -147,10 +147,10 @@
     <child link="left_arm_mount" />
     <parent link="base_link" />
-    <origin xyz="-0.020 0.184 1.1384" rpy="0 0 0" />
+    <origin xyz="-0.020 0.184 1.1384" rpy="0 0 1.5707" />
   </joint>
   <joint name="right_arm_attach" type="fixed">
     <child link="right_arm_mount" />
     <parent link="base_link" />
-    <origin xyz="-0.020 -0.184 1.1384" rpy="0 0 0" />
+    <origin xyz="-0.020 -0.184 1.1384" rpy="0 0 1.5707" />
   </joint>
  <!-- PTU

Commit message: Fixed robot_mass joint

File: description/urdf/pioneer-lx-devil.urdf (robot description, URDF)
Before this commit: robot pioneer-lx-devil, 37 links, 36 joints
Links:
- added link robot_mass, mass 57.8
- link base_link: mass 57.8 -> None
Joints:
- removed joint left_jaco_joint_5
- removed joint left_jaco_joint_6
- removed joint right_jaco_joint_5
- removed joint right_jaco_joint_6
- added joint left_jaco2_joint_5: type continuous, parent left_jaco2_link_4, child left_jaco2_link_5, origin xyz=0.03700 0 -0.06408 rpy=0 -1.0471975512 0, axis 0 0 -1, limit lower=-6.28318530718 upper=6.28318530718 effort=30 velocity=0.35
- added joint left_jaco2_joint_6: type continuous, parent left_jaco2_link_5, child left_jaco2_link_hand, origin xyz=0.03700 0 -0.06408 rpy=-1.0471975512 0 1.57079632679, axis 0 0 -1, limit lower=-6.28318530718 upper=6.28318530718 effort=30 velocity=0.35
- added joint right_jaco2_joint_5: type continuous, parent right_jaco2_link_4, child right_jaco2_link_5, origin xyz=0.03700 0 -0.06408 rpy=0 -1.0471975512 0, axis 0 0 -1, limit lower=-6.28318530718 upper=6.28318530718 effort=30 velocity=0.35
- added joint right_jaco2_joint_6: type continuous, parent right_jaco2_link_5, child right_jaco2_link_hand, origin xyz=0.03700 0 -0.06408 rpy=-1.0471975512 0 1.57079632679, axis 0 0 -1, limit lower=-6.28318530718 upper=6.28318530718 effort=30 velocity=0.35
- added joint robot_mass_attach: type fixed, parent base_link, child robot_mass

File: description/urdf/pioneer-lx-devil.urdf.xacro (robot description, xacro)
@@ -29,7 +29,7 @@
     </inertial>
   </link>
-  <joint name="base_link_mass_attach">
+  <joint name="robot_mass_attach" type="fixed">
     <parent link="base_link" />
-    <child link="base_link_mass" />
+    <child link="robot_mass" />
   </joint>
   <!-- right wheel -->

Commit message: Moved arm mounting position to top mounting holes, use properties in xacro for easier modification.

File: description/urdf/pioneer-lx-devil.urdf (robot description, URDF)
Before this commit: robot pioneer-lx-devil, 38 links, 37 joints
Joints:
- joint left_arm_attach: origin xyz=-0.020 0.184 1.1384 rpy=0 0 1.5707 -> xyz=-0.02 0.184 1.086 rpy=0 0 1.5707
- joint left_jaco2_joint_2: limit lower=-3.14159265359 upper=0.0 effort=30 velocity=0.35 -> lower=-3.14159265359 upper=0 effort=30 velocity=0.35
- joint right_arm_attach: origin xyz=-0.020 -0.184 1.1384 rpy=0 0 1.5707 -> xyz=-0.02 -0.184 1.086 rpy=0 0 1.5707
- joint right_jaco2_joint_2: limit lower=-3.14159265359 upper=0.0 effort=30 velocity=0.35 -> lower=-3.14159265359 upper=0 effort=30 velocity=0.35

File: description/urdf/pioneer-lx-devil.urdf.xacro (robot description, xacro)
@@ -3,4 +3,21 @@
   <!-- TODO share pioneer lx mobile robot components with pioneer-lx urdf by
 including macro. -->
+  <property name="deck_height" value="0.076" />
+  <property name="deck_width" value="0.437" />
+  <property name="deck_length" value="0.407" />
+  <property name="base_height" value="0.35" />
+  <property name="base_width" value="0.50" />
+  <property name="base_length" value="0.697" />
+  <property name="plinth_width" value="0.5" />
+  <property name="plinth_length" value="0.697" /> <!-- at bottom -->
+  <property name="plinth_height" value="0.99" />
+  <property name="plinth_bottom_mount_holes_z" value="0.584" />
+  <property name="plinth_middle_mount_holes_z" value="0.73" />
+  <property name="plinth_top_mount_holes_z" value="${plinth_height - 0.03}" />
+  <property name="arm_mount_offset_z" value="0.076" />   <!-- height of bottom of jaco arm above mounting hole when mounted using supplied 8020 hardware fixtrue -->
+  <property name="arm_mount_holes_z" value="${plinth_bottom_mount_holes_z}" /> <!-- change this if you move the arm mounting to one of the other sets of holes -->
+  <property name="arm_origin_z" value="${base_height + deck_height + arm_mount_holes_z + arm_mount_offset_z}" />
+  <property name="left_arm_origin" value="-0.02 0.184 ${arm_origin_z}" /> <!-- old z was 1.1384 -->
+  <property name="right_arm_origin" value="-0.02 -0.184 ${arm_origin_z}" />
   <link name="base_link">
     <!-- base_link origin point is center of rotation, on the floor. -->
@@ -17,5 +34,6 @@
     <collision name="base_link_collision">
       <geometry name="base_link_collision_geom">
-        <box size="0.697 0.5 0.35" />
+        <box size="${base_length} ${base_width} ${base_height}" />
+        <!-- box size="0.697 0.5 0.35" / -->
       </geometry>
       <origin xyz="0 0 0.200" rpy="0 0 0" />
@@ -97,5 +115,5 @@
     <visual name="deck_visual">
       <geometry name="deck_visual_geom">
-        <box size="0.407 0.437 0.076" />
+        <box size="${deck_length} ${deck_width} ${deck_height}" />
       </geometry>
       <material name="lx_deck_mat">
@@ -105,5 +123,6 @@
     <collision name="deck_collision">
       <geometry name="deck_collision_geom">
-        <box size="0.407 0.437 0.076" />
+        <box size="${deck_length} ${deck_width} ${deck_height}" />
+        <!-- box size="0.407 0.437 0.076" / -->
       </geometry>
     </collision>
@@ -154,10 +173,12 @@
     <child link="left_arm_mount" />
     <parent link="base_link" />
-    <origin xyz="-0.020 0.184 1.1384" rpy="0 0 1.5707" />
+    <origin xyz="${left_arm_origin}" rpy="0 0 1.5707" />
+    <!-- old z was 1.1384 -->
   </joint>
   <joint name="right_arm_attach" type="fixed">
     <child link="right_arm_mount" />
     <parent link="base_link" />
-    <origin xyz="-0.020 -0.184 1.1384" rpy="0 0 1.5707" />
+    <origin xyz="${right_arm_origin}" rpy="0 0 1.5707" />
+    <!-- old z was 1.1384 -->
   </joint>
  <!-- PTU

Commit message: add seekurjr and terabot arm, misc fixes, rename item in pioneer-lx-devil so depthimage_to_laserscan can be used

File: description/urdf/pioneer-lx-devil.urdf (robot description, URDF)
Before this commit: robot pioneer-lx-devil, 38 links, 37 joints
Links:
- added link camera_depth_frame, mass 0.0
Joints:
- added joint camera_depth_frame_joint: type fixed, parent kinect, child camera_depth_frame, origin xyz=0 0 0

File: description/urdf/pioneer-lx-devil.urdf.xacro (robot description, xacro)
@@ -217,3 +217,16 @@
     <origin xyz="0 0 0.0325" />
   </joint>
+  <!-- hack for depthimage_to_laserscan (todo: configure depthimage_to_laserscan to use "kinect" as frame -->
+  <link name="camera_depth_frame">
+    <origin xyz="0 0 0" />
+    <inertial>
+      <mass value="0.0" />
+      <inertia ixx="1" ixy="0" ixz="0" iyy="1" iyz="0" izz="1" />
+    </inertial>
+  </link>
+  <joint name="camera_depth_frame_joint" type="fixed">
+    <parent link="kinect" />
+    <child link="camera_depth_frame" />
+    <origin xyz="0 0 0" />
+  </joint>
 </robot>
