Commit message: Modified some friction parameters and other minor changes

File: description/urdf/pioneer3at.urdf (robot description, URDF)
Before this commit: robot pioneer3at, 16 links, 15 joints
Links:
- link base_link: mass 10.0 -> 15.0
Joints:
- removed joint bp3at_back_left_axle_joint
- removed joint bp3at_back_right_axle_joint
- added joint p3at_back_left_axle_joint: type fixed, parent base_link, child p3at_back_left_axle, origin xyz=-0.134 0.156 0.111 rpy=0 0 0
- added joint p3at_back_right_axle_joint: type fixed, parent base_link, child p3at_back_right_axle, origin xyz=-0.134 -0.156 0.111 rpy=0 0 0

File: description/urdf/pioneer3at.urdf.xacro (robot description, xacro)
@@ -8,5 +8,5 @@
 	<link name="base_link">
 		<inertial>
-			<mass value="10.0"/>
+			<mass value="15.0"/>
 			<origin xyz="0 0 0.177"/>
 			<inertia ixx="0.3338" ixy="0.0" ixz="0.0"
@@ -59,5 +59,5 @@
 	</link>
 	<gazebo reference="top_plate">
-		<material value="Gazebo/Black"/>
+    <material>Gazebo/Black</material>
 	</gazebo>
 	<joint name="base_top_joint" type="fixed">
@@ -256,5 +256,5 @@
 		<material value="Gazebo/Grey"/>
 	</gazebo>
-	<joint name="bp3at_back_${side}_axle_joint" type="fixed">
+	<joint name="p3at_back_${side}_axle_joint" type="fixed">
 		<origin xyz="-0.134 ${reflect*0.156} 0.111" rpy="0 0 0"/>
 		<parent link="base_link"/>
@@ -327,6 +327,10 @@
     <kp>1000000.0</kp> <!-- kp and kd for rubber -->
     <kd>100.0</kd>
-    <mu1>10.0</mu1>
+    <mu1>1.0</mu1> <!-- was 10 -->
     <mu2>1.0</mu2>
+      <!-- how to get these into <surface><friction><ode>... ?
+        slip1 0.5 /slip1
+         slip2 0 /slip2
+      -->
     <fdir1>0 1 0</fdir1> <!-- is this correct? -->
     <maxVel>1.0</maxVel>
@@ -337,6 +341,10 @@
     <kp>1000000.0</kp> <!-- kp and kd for rubber -->
     <kd>100.0</kd>
-    <mu1>10.0</mu1>
+    <mu1>1.0</mu1> <!-- was 10 -->
     <mu2>1.0</mu2>
+      <!-- how to get these into <surface><friction><ode>... ?
+        slip1 0.5 /slip1
+         slip2 0 /slip2
+      -->
     <fdir1>0 1 0</fdir1> <!-- is this correct? -->
     <maxVel>1.0</maxVel>
@@ -357,4 +365,5 @@
     <wheelDiameter>0.215</wheelDiameter>
     <robotBaseFrame>base_link</robotBaseFrame>
+    <MaxForce>5.0</MaxForce>
     <torque>200</torque>
     <commandTopic>cmd_vel</commandTopic>

File: description/urdf/pioneer3dx.urdf.xacro (robot description, xacro)
@@ -52,5 +52,6 @@
 	</link>
 	<gazebo reference="top_plate">
-		<material value="Gazebo/Black"/>
+		<!-- material value="Gazebo/Black"/ -->
+		<material>Gazebo/Black</material>
 	</gazebo>
     <joint name="base_top_joint" type="fixed">

Commit message: P3AT was too light. Add correct weight with 3 batteries.

File: description/urdf/pioneer3at.urdf (robot description, URDF)
Before this commit: robot pioneer3at, 16 links, 15 joints
Links:
- link base_link: mass 10.0 -> 21.5
- link p3at_back_left_wheel: mass 0.5 -> 1.2
- link p3at_back_right_wheel: mass 0.5 -> 1.2
- link p3at_front_left_wheel: mass 0.5 -> 1.2
- link p3at_front_right_wheel: mass 0.5 -> 1.2

File: description/urdf/pioneer3at.urdf.xacro (robot description, xacro)
@@ -7,10 +7,17 @@
 <!-- Chassis -->
 	<link name="base_link">
-		<inertial>
-			<mass value="10.0"/>
-			<origin xyz="0 0 0.177"/>
-			<inertia ixx="0.3338" ixy="0.0" ixz="0.0"
-				 iyy="0.4783" iyz="0.0"
-				 izz="0.3338"/>
+		<!--  For pointers on inertial and gazebo-related parameters see
+		       * http://wiki.ros.org/urdf/Tutorials/Adding%20Physical%20and%20Collision%20Properties%20to%20a%20URDF%20Model
+                       * http://answers.gazebosim.org/question/4372/the-inertia-matrix-explained/
+		       * http://gazebosim.org/tutorials?tut=inertia&cat=build_robot, and
+                       * http://gazebosim.org/tutorials/?tut=ros_urdf
+                       * http://en.wikipedia.org/wiki/List_of_moment_of_inertia_tensors
+                -->
+		<inertial>
+			<mass value="21.5"/> <!-- P3AT 18.6kg plus three batteries @ 2.4kg each  minus four wheels @ 1.4 kg ea and top plate @ 0.1 kg-->
+			<origin xyz="0 -0.1 0.177"/>
+			<inertia ixx="0.3338" ixy="0.0"     ixz="0.0"
+				              iyy="0.4783"  iyz="0.0"
+				                            izz="0.3338"/>
 		</inertial>
 		<visual name="base_visual">
@@ -195,5 +202,5 @@
 	<link name="p3at_front_${side}_wheel">
 		<inertial>
-			<mass value="0.5"/>
+			<mass value="1.2"/> <!-- 1.4 kg - axle 0.1 kg - hub 0.1 kg -->
 			<origin xyz="0 0 0"/>
 			<inertia ixx="0.012411765597" ixy="0" ixz="0"
@@ -292,8 +299,9 @@
 	<link name="p3at_back_${side}_wheel">
 		<inertial>
-			<mass value="0.5"/>
+			<mass value="1.2"/>
 			<origin xyz="0 0 0"/>
 			<inertia ixx="0.012411765597" ixy="0" ixz="0"
-         iyy="0.015218160428" iyz="0" izz="0.011763977943"/>
+                                                      iyy="0.015218160428" iyz="0"
+                                                                           izz="0.011763977943"/>
       </inertial>
 	<visual name="base_visual">
@@ -324,4 +332,5 @@
 		<child link="p3at_back_${side}_wheel"/>
 	</joint>
+  <!-- see http://gazebosim.org/tutorials/?tut=ros_urdf -->
   <gazebo reference="p3at_back_${side}_wheel">
     <kp>1000000.0</kp> <!-- kp and kd for rubber -->
@@ -358,7 +367,7 @@
     <robotBaseFrame>base_link</robotBaseFrame>
     <torque>200</torque>
-    <commandTopic>sim_p3at/cmd_vel</commandTopic>
-    <odometryTopic>sim_p3at/odom</odometryTopic>
-    <odometryFrame>sim_p3at/odom</odometryFrame>
+    <commandTopic>cmd_vel</commandTopic>
+    <odometryTopic>odom</odometryTopic>
+    <odometryFrame>odom</odometryFrame>
     <broadcastTF>1</broadcastTF>
   </plugin>

Commit message: fixed some issuses with Jessie/gazebo7

File: description/urdf/pioneer3at.urdf (robot description, URDF)
Before this commit: robot pioneer3at, 16 links, 15 joints
Links:
- link back_sonar: geometry collision box size=0.1 0.1 0.1; visual mesh filename=package://amr_robots_description/meshes/p3at_meshes/back_so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
- link front_sonar: geometry collision box size=0.1 0.1 0.1; visual mesh filename=package://amr_robots_description/meshes/p3at_meshes/front_s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
- link p3at_front_left_axle: geometry collision box size=0.1 0.1 0.1; visual mesh filename=package://amr_robots_description/meshes/p3at_meshes/axle.stl
- link p3at_front_left_hub: geometry collision box size=0.1 0.1 0.1; visual mesh filename=package://amr_robots_description/meshes/p3at_meshes/left_hu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
- link p3at_front_right_axle: geometry collision box size=0.1 0.1 0.1; visual mesh filename=package://amr_robots_description/meshes/p3at_meshes/axle.stl
- link p3at_front_right_hub: geometry collision box size=0.1 0.1 0.1; visual mesh filename=package://amr_robots_description/meshes/p3at_meshes/right_h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
- link top_plate: geometry collision box size=0.1 0.1 0.1; visual mesh filename=package://amr_robots_description/meshes/p3at_meshes/top.stl

File: description/urdf/pioneer3at.urdf.xacro (robot description, xacro)
@@ -61,5 +61,5 @@
 			<origin xyz="0 0 0" rpy="0 0 0"/>
 			<geometry>
-				<box size="0 0 0"/>
+				<box size="0.1 0.1 0.1"/>
 			</geometry>
 		</collision>
@@ -93,5 +93,5 @@
 			<origin xyz="0 0 0" rpy="0 0 0"/>
 			<geometry>
-				<box size="0 0 0"/>
+				<box size="0.1 0.1 0.1"/>
 			</geometry>
 		</collision>
@@ -124,5 +124,5 @@
 			<origin xyz="0 0 0" rpy="0 0 0"/>
 			<geometry>
-				<box size="0 0 0"/>
+				<box size="0.1 0.1 0.1"/>
 			</geometry>
 		</collision>
@@ -157,5 +157,5 @@
 		<origin xyz="0 0 0" rpy="0 0 0"/>
 		<geometry>
-			<box size="0 0 0"/>
+			<box size="0.1 0.1 0.1"/>
 		</geometry>
 	</collision>
@@ -188,5 +188,5 @@
 		<origin xyz="0 0 0" rpy="0 0 0"/>
 		<geometry>
-			<box size="0 0 0"/>
+			<box size="0.1 0.1 0.1"/>
 		</geometry>
 	</collision>

File: description/urdf/pioneer3at_body.xacro (robot description, xacro)
@@ -54,5 +54,5 @@
 			<origin xyz="0 0 0" rpy="0 0 0"/>
 			<geometry>
-				<box size="0 0 0"/>
+				<box size="0.1 0.1 0.1"/>
 			</geometry>
 		</collision>
@@ -86,5 +86,5 @@
 			<origin xyz="0 0 0" rpy="0 0 0"/>
 			<geometry>
-				<box size="0 0 0"/>
+				<box size="0.1 0.1 0.1"/>
 			</geometry>
 		</collision>
@@ -117,5 +117,5 @@
 			<origin xyz="0 0 0" rpy="0 0 0"/>
 			<geometry>
-				<box size="0 0 0"/>
+				<box size="0.1 0.1 0.1"/>
 			</geometry>
 		</collision>
@@ -150,5 +150,5 @@
 		<origin xyz="0 0 0" rpy="0 0 0"/>
 		<geometry>
-			<box size="0 0 0"/>
+			<box size="0.1 0.1 0.1"/>
 		</geometry>
 	</collision>
@@ -181,5 +181,5 @@
 		<origin xyz="0 0 0" rpy="0 0 0"/>
 		<geometry>
-			<box size="0 0 0"/>
+			<box size="0.1 0.1 0.1"/>
 		</geometry>
 	</collision>

File: description/urdf/pioneer3dx.urdf (robot description, URDF)
Before this commit: robot pioneer3dx, 11 links, 10 joints
Links:
- link back_sonar: geometry collision box size=0.1 0.1 0.1; visual mesh filename=package://amr_robots_description/meshes/p3dx_meshes/back_so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
- link caster_swivel: geometry collision box size=0.1 0.1 0.1; visual mesh filename=package://amr_robots_description/meshes/p3dx_meshes/caster_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
- link front_sonar: geometry collision box size=0.1 0.1 0.1; visual mesh filename=package://amr_robots_description/meshes/p3dx_meshes/front_s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

File: description/urdf/pioneer3dx.urdf.xacro (robot description, xacro)
@@ -80,5 +80,5 @@
 			<origin xyz="0 0 0" rpy="0 0 0"/>
 			<geometry>
-				<box size="0 0 0"/>
+				<box size="0.1 0.1 0.1"/>
 			</geometry>
 		</collision>
@@ -116,5 +116,5 @@
 			<origin xyz="0 0 0" rpy="0 0 0"/>
 			<geometry>
-				<box size="0 0 0"/>
+				<box size="0.1 0.1 0.1"/>
 			</geometry>
 		</collision>
@@ -148,5 +148,5 @@
 		<origin xyz="0 0 0" rpy="0 0 0"/>
 		<geometry>
-			<box size="0 0 0"/>
+			<box size="0.1 0.1 0.1"/>
 		</geometry>
 	</collision>

File: description/urdf/pioneer3dx_body.xacro (robot description, xacro)
@@ -91,5 +91,5 @@
 		<origin xyz="0 0 0" rpy="0 0 0"/>
 		<geometry>
-			<box size="0 0 0"/>
+			<box size="0.1 0.1 0.1"/>
 		</geometry>
 	</collision>
@@ -275,5 +275,5 @@
 			<origin xyz="0 0 0" rpy="0 0 0"/>
 			<geometry>
-				<box size="0 0 0"/>
+				<box size="0.1 0.1 0.1"/>
 			</geometry>
 		</collision>

File: description/urdf/pioneer3dx_orig.2.xacro (robot description, xacro)
@@ -49,5 +49,5 @@
         <origin xyz="0 0 0" rpy="0 0 0"/>
         <geometry>
-          <box size="0 0 0"/>
+          <box size="0.1 0.1 0.1"/>
         </geometry>
       </collision>
@@ -73,5 +73,5 @@
         <origin xyz="0 0 0" rpy="0 0 0"/>
         <geometry>
-          <box size="0 0 0"/>
+          <box size="0.1 0.1 0.1"/>
         </geometry>
       </collision>
@@ -97,5 +97,5 @@
         <origin xyz="0 0 0" rpy="0 0 0"/>
         <geometry>
-          <box size="0 0 0"/>
+          <box size="0.1 0.1 0.1"/>
         </geometry>
       </collision>
@@ -121,5 +121,5 @@
         <origin xyz="0 0 0" rpy="0 0 0"/>
         <geometry>
-          <box size="0 0 0"/>
+          <box size="0.1 0.1 0.1"/>
         </geometry>
       </collision>
@@ -145,5 +145,5 @@
         <origin xyz="0 0 0" rpy="0 0 0"/>
         <geometry>
-          <box size="0 0 0"/>
+          <box size="0.1 0.1 0.1"/>
         </geometry>
       </collision>
@@ -169,5 +169,5 @@
         <origin xyz="0 0 0" rpy="0 0 0"/>
         <geometry>
-          <box size="0 0 0"/>
+          <box size="0.1 0.1 0.1"/>
         </geometry>
       </collision>
@@ -193,5 +193,5 @@
         <origin xyz="0 0 0" rpy="0 0 0"/>
         <geometry>
-          <box size="0 0 0"/>
+          <box size="0.1 0.1 0.1"/>
         </geometry>
       </collision>

File: description/urdf/pioneer3dx_wheel.xacro (robot description, xacro)
@@ -60,5 +60,5 @@
     <origin xyz="0 0 0" rpy="0 0 0"/>
     <geometry>
-      <box size="0 0 0"/>
+      <box size="0.1 0.1 0.1"/>
     </geometry>
   </collision>

Commit message: updated urdf

File: description/urdf/pioneer3at.urdf (robot description, URDF)
Before this commit: robot pioneer3at, 16 links, 15 joints
Links:
- added link imu_link, mass 0.001; collision box size=.001 .001 .001; visual box size=0.001 0.001 0.001
Joints:
- added joint imu_joint: type fixed, parent base_link, child imu_link, origin xyz=0 0 0.19, axis 1 0 0

File: description/urdf/pioneer3at.urdf.xacro (robot description, xacro)
@@ -5,4 +5,5 @@
        xmlns:xacro="http://ros.org/wiki/xacro"
 name="pioneer3at">
+<xacro:include filename="$(find amr_robots_description)/urdf/materials.xacro" />
 <!-- Chassis -->
 	<link name="base_link">
@@ -38,6 +39,42 @@
 	</link>
 	<gazebo reference="base_link">
-		<material value="Gazebo/Red"/>
-	</gazebo>
+      <material>
+         <!--
+      <script>
+         <uri>/usr/share/gazebo-7/media/materials/scripts/gazebo.material</uri>
+          <name>Gazebo/Green</name>
+      </script>
+-->
+          <ambient>1 0 0 0</ambient>
+          <diffuse>1 0 0 0</diffuse>
+          <specular>0 0 0 1</specular>
+          <emissive>0 0 0 1</emissive>
+</material>
+	</gazebo>
+  <joint name="imu_joint" type="fixed">
+    <axis xyz="1 0 0"/> <!-- 0 1 0 -->
+    <origin xyz="0 0 0.19"/>
+    <parent link="base_link"/>
+    <child link="imu_link"/>
+  </joint>
+<link name="imu_link">
+  <inertial>
+    <mass value="0.001"/>
+    <origin rpy="0 0 0" xyz="0 0 0"/>
+    <inertia ixx="0.0001" ixy="0" ixz="0" iyy="0.000001" iyz="0" izz="0.0001"/>
+  </inertial>
+  <visual>
+    <origin rpy="0 0 0" xyz="0 0 0"/>
+    <geometry>
+      <box size="0.001 0.001 0.001"/>
+    </geometry>
+  </visual>
+  <collision>
+    <origin rpy="0 0 0" xyz="0 0 0"/>
+    <geometry>
+      <box size=".001 .001 .001"/>
+    </geometry>
+  </collision>
+</link>
 <!-- Top -->
 	<link name="top_plate">
@@ -364,4 +401,12 @@
 <xacro:macro name="p3at_gazebo_ext">
 <gazebo>
+    <plugin name="imu_plugin" filename="libgazebo_ros_imu.so">
+        <alwaysOn>true</alwaysOn>
+        <bodyName>imu_link</bodyName>
+        <topicName>imu_data</topicName>
+        <serviceName>imu_service</serviceName>
+        <gaussianNoise>0.0</gaussianNoise>
+        <updateRate>30.0</updateRate>
+    </plugin>
   <plugin name="skid_steer_drive_controller" filename="libgazebo_ros_skid_steer_drive.so">
     <updateRate>100.0</updateRate>
@@ -381,4 +426,10 @@
     <broadcastTF>1</broadcastTF>
   </plugin>
+  <plugin name="ground_truth" filename="libgazebo_ros_p3d.so">
+    <frameName>map</frameName>
+    <bodyName>base_link</bodyName>
+    <topicName>odom_gt</topicName>
+    <updateRate>30.0</updateRate>
+  </plugin>
 </gazebo>
 </xacro:macro>
