Commit message: adding working P3DX and P3AT urdfs.

File: description/urdf/pioneer3at.urdf.xacro (robot description, xacro)
@@ -4,5 +4,5 @@
        xmlns:interface="http://playerstage.sourceforge.net/gazebo/xmlschema/#interface"
        xmlns:xacro="http://ros.org/wiki/xacro"
->
+name="pioneer3at">
 <!-- Chassis -->
 	<link name="base_link">
@@ -359,4 +359,8 @@
   </plugin>
 </gazebo>
-</xacro:macro>
+<xacro:p3at_front suffix="left" reflect="1"/>
+<xacro:p3at_front suffix="right" reflect="-1"/>
+<xacro:p3at_back suffix="left" reflect="1"/>
+<xacro:p3at_back suffix="right" reflect="-1"/>
+<xacro:p3at_gazebo_ext/>
 </robot>

File: description/urdf/pioneer3dx.urdf.xacro (robot description, xacro)
@@ -5,6 +5,6 @@
 	xmlns:interface="http://playerstage.sourceforge.net/gazebo/xmlschema/#interface"
 	xmlns:xacro="http://ros.org/wiki/xacro">
-  <!--<include filename="$(find p2os_urdf)/defs/materials.xacro"/>-->
-  <include filename="$(find p2os_urdf)/defs/pioneer3dx_wheel.xacro"/>
+  <!--<include filename="$(find amr_robots_description)/urdf/materials.xacro"/>-->
+  <xacro:include filename="$(find amr_robots_description)/urdf/pioneer3dx_wheel.xacro"/>
 <!-- Chassis -->
 	<link name="base_link">
@@ -20,5 +20,5 @@
 			<origin xyz="-0.045 0 0.148" rpy="0 0 0"/>
 			<geometry name="pioneer_geom">
-				<mesh filename="package://p2os_urdf/meshes/p3dx_meshes/chassis.stl"/>
+				<mesh filename="package://amr_robots_description/meshes/p3dx_meshes/chassis.stl"/>
 			</geometry>
 			<material name="ChassisRed">
@@ -33,13 +33,7 @@
 		</collision>
 	</link>
-    <joint name="base_top_joint" type="fixed">
-		<origin xyz="-0.045 0 0.234" rpy="0 0 0"/>
-		<axis xzy="0 0 1"/>
-		<parent link="base_link"/>
-		<child link="top_plate"/>
-	</joint>
-	<link name="base_top">
-		<inertial>
-			<mass value="0"/>
+	<link name="top_plate">
+		<inertial>
+			<mass value="0.01"/>
 			<origin xyz="0 0 0"/>
 			<inertia ixx="1" ixy="0" ixz="0"
@@ -47,8 +41,8 @@
  				izz="1"/>
 		</inertial>
-		<visual>
+		<visual name="pioneer_geom">
 			<origin xyz="0 0 0" rpy="0 0 0"/>
 			<geometry name="pioneer_geom">
-				<mesh filename="package://p2os_urdf/meshes/p3dx_meshes/top.stl"/>
+				<mesh filename="package://amr_robots_description/meshes/p3dx_meshes/top.stl"/>
 			</geometry>
 			<material name="TopBlack">
@@ -56,25 +50,95 @@
 			</material>
 		</visual>
-		<collision>
-			<origin xyz="0 0 0" rpy="0 0 0"/>
-			<geometry>
-				<box size="0 0 0"/>
-			</geometry>
-		</collision>
-	</link>
-<!-- Swivel -->
-	<link name="swivel">
-		<inertial>
-			<mass value="0"/>
+	</link>
+	<gazebo reference="top_plate">
+		<material value="Gazebo/Black"/>
+	</gazebo>
+    <joint name="base_top_joint" type="fixed">
+		<origin xyz="-0.045 0 0.234" rpy="0 0 0"/>
+		<axis xzy="0 0 1"/>
+		<parent link="base_link"/>
+		<child link="top_plate"/>
+	</joint>
+	<link name="front_sonar">
+		<inertial>
+			<mass value="0.0001"/>
 			<origin xyz="0 0 0"/>
 			<inertia ixx="1" ixy="0" ixz="0"
 				 iyy="1" iyz="0" izz="1"/>
+		</inertial>
+		<visual name="pioneer_geom">
+			<origin xyz="0 0 0" rpy="0 0 0"/>
+			<geometry name="pioneer_geom">
+				<mesh filename="package://amr_robots_description/meshes/p3dx_meshes/front_sonar.stl"/>
+			</geometry>
+			<material name="SonarYellow">
+				<color rgba="0.715 0.583 0.210 1.0"/>
+			</material>
+		</visual>
+		<collision>
+			<origin xyz="0 0 0" rpy="0 0 0"/>
+			<geometry>
+				<box size="0 0 0"/>
+			</geometry>
+		</collision>
+	</link>
+	<gazebo reference="front_sonar">
+		<material value="Gazebo/Yellow"/>
+	</gazebo>
+	<joint name="base_front_joint" type="fixed">
+		<origin xyz="-0.198 0 0.208" rpy="0 0 0"/>
+		<parent link="base_link"/>
+		<child link="front_sonar"/>
+	</joint>
+	<joint name="base_back_joint" type="fixed">
+		<origin xyz="0.109 0 0.209" rpy="0 0 0"/>
+		<parent link="base_link"/>
+		<child link="back_sonar"/>
+	</joint>
+	<link name="back_sonar">
+		<inertial>
+			<mass value="0"/>
+			<origin xyz="0 0 0"/>
+			<inertia ixx="1" ixy="0" ixz="0"
+				 iyy="1" iyz="0" izz="1"/>
+		</inertial>
+		<visual name="base_visual">
+			<origin xyz="0 0 0" rpy="0 0 0"/>
+			<geometry name="pioneer_geom">
+				<mesh filename="package://amr_robots_description/meshes/p3dx_meshes/back_sonar.stl"/>
+			</geometry>
+			<material name="SonarYellow">
+				<color rgba="0.715 0.583 0.210 1.0"/>
+			</material>
+		</visual>
+		<collision>
+			<origin xyz="0 0 0" rpy="0 0 0"/>
+			<geometry>
+				<box size="0 0 0"/>
+			</geometry>
+		</collision>
+	</link>
+	<!-- Caster -->
+	<joint name="base_caster_swivel_joint" type="continuous">
+		<origin xyz="-0.185 0 0.055" rpy="0 0 0"/>
+		<anchor xyz="0 0 0"/>
+    	<limit effort="100" velocity="100" k_velocity="0" />
+    	<joint_properties damping="0.0" friction="0.0" />
+		<parent link="base_link"/>
+		<child link="caster_swivel"/>
+	</joint>
+	<link name="caster_swivel">
+		<inertial>
+			<mass value="0.1"/>
+			<origin xyz="0 0 0"/>
+			<inertia ixx="0.01" ixy="0" ixz="0"
+				 iyy="0.01" iyz="0" izz="0.01"/>
   	 	</inertial>
-	<visual name="base_visual">
+	<visual name="pioneer_geom">
 		<origin xyz="0 0 0" rpy="0 0 0"/>
 		<geometry name="pioneer_geom">
-			<mesh filename="package://p2os_urdf/meshes/p3dx_meshes/swivel.stl"/>
-		</geometry>
-		<material name="swivel">
+			<mesh filename="package://amr_robots_description/meshes/p3dx_meshes/caster_swivel.stl"/>
+		</geometry>
+		<material name="caster_swivel">
 			<color rgba="0.5 0.5 0.5 1"/>
 		</material>
@@ -87,27 +151,21 @@
 	</collision>
 	</link>
- 	<joint name="base_swivel_joint" type="continuous">
-		<origin xyz="-0.185 0 0.055" rpy="0 0 0"/>
-		<axis xyz="0 0 1" />
-		<anchor xyz="0 0 0" />
-		<limit effort="100" velocity="100" />
-		<joint_properties damping="0.0" friction="0.0" />
-		<parent link="base_link"/>
-		<child link="swivel"/>
-	</joint>
+	<gazebo reference="caster_swivel">
+		<material value="Gazebo/Grey"/>
+	</gazebo>
 <!-- Center Wheel + Hubcap -->
-	<link name="center_hubcap">
-		<inertial>
-			<mass value="0"/>
-			<origin xyz="0 0 0"/>
-			<inertia ixx="1" ixy="0" ixz="0"
-				 iyy="1" iyz="0" izz="1"/>
+	<link name="caster_hubcap">
+		<inertial>
+			<mass value="0.01"/>
+			<origin xyz="0 0 0"/>
+			<inertia ixx="0.012411765597" ixy="-0.000711733678" ixz="0.00050272983"
+				 iyy="0.015218160428" iyz="-0.000004273467" izz="0.011763977943"/>
   	 	</inertial>
-	<visual name="base_visual">
+	<visual name="pioneer_geom">
 		<origin xyz="0 0 0" rpy="0 0 0"/>
 		<geometry name="pioneer_geom">
-			<mesh filename="package://p2os_urdf/meshes/p3dx_meshes/center_hubcap.stl"/>
-		</geometry>
-		<material name="swivel">
+			<mesh filename="package://amr_robots_description/meshes/p3dx_meshes/caster_hubcap.stl"/>
+		</geometry>
+		<material name="caster_swivel">
 			<color rgba="0.5 0.5 0.5 1"/>
 		</material>
@@ -116,28 +174,31 @@
 		<origin xyz="0 0 0" rpy="0 0 0"/>
 		<geometry>
-			<box size="0 0 0"/>
+			<box size="0.05 0.05 0.05"/>
 		</geometry>
 	</collision>
 	</link>
-	<joint name="swivel_hubcap_joint" type="continuous">
+	<gazebo reference="caster_hubcap">
+		<material value="Gazebo/Grey"/>
+	</gazebo>
+	<joint name="caster_swivel_hubcap_joint" type="continuous">
 		<origin xyz="-0.026 0 -0.016" rpy="0 0 0"/>
-		<axis xyz="0 1 0" />
-		<anchor xyz="0 0 0" />
-		<limit effort="100" velocity="100" />
-		<joint_properties damping="0.0" friction="0.0" />
-		<parent link="swivel"/>
-		<child link="center_hubcap"/>
-	</joint>
-	<link name="center_wheel">
-		<inertial>
-			<mass value="0"/>
-			<origin xyz="0 0 0"/>
-			<inertia ixx="1" ixy="0" ixz="0"
-				 iyy="1" iyz="0" izz="1"/>
+		<axis xyz="0 1 0"/>
+		<anchor xyz="0 0 0"/>
+    <limit effort="100" velocity="100" k_velocity="0" />
+    <joint_properties damping="0.0" friction="0.0" />
+	  <parent link="caster_swivel"/>
+		<child link="caster_wheel"/>
+	</joint>
+	<link name="caster_wheel">
+		<inertial>
+			<mass value="0.1"/>
+			<origin xyz="0 0 0"/>
+			<inertia ixx="0.012411765597" ixy="-0.000711733678" ixz="0.00050272983"
+				 iyy="0.015218160428" iyz="-0.000004273467" izz="0.011763977943"/>
   	 	</inertial>
-	<visual name="base_visual">
+	<visual name="pioneer_geom">
 		<origin xyz="0 0 0" rpy="0 0 0"/>
 		<geometry name="pioneer_geom">
-			<mesh filename="package://p2os_urdf/meshes/p3dx_meshes/center_wheel.stl"/>
+			<mesh filename="package://amr_robots_description/meshes/p3dx_meshes/caster_wheel.stl"/>
 		</geometry>
 		<material name="WheelBlack">
@@ -146,74 +207,108 @@
 	</visual>
 	<collision>
-		<origin xyz="0 0 0" rpy="0 0 0"/>
+		<origin xyz="0 0 0" rpy="${-3.1415927/2.0} 0 0"/>
 		<geometry>
-			<box size="0 0 0"/>
+			<!--<mesh filename="package://amr_robots_description/meshes/p3dx_meshes/caster_wheel.stl"/>-->
+			<cylinder radius="0.0375" length="0.01"/>
 		</geometry>
 	</collision>
 	</link>
-	<joint name="center_wheel_joint" type="fixed">
+	<gazebo reference="left_hub">
+		<material value="Gazebo/Yellow"/>
+	</gazebo>
+	<joint name="caster_wheel_joint" type="fixed">
 		<origin xyz="-0.0035 0 -0.001" rpy="0 0 0"/>
-		<parent link="center_hubcap"/>
-		<child link="center_wheel"/>
-	</joint>
-<xacro:p3dx_wheel suffix="left" reflect="1"/>
-<xacro:p3dx_wheel suffix="right" reflect="-1"/>
-<!-- Front + Back Sonar -->
-	<link name="front_sonar">
-		<inertial>
-			<mass value="0"/>
-			<origin xyz="0 0 0"/>
-			<inertia ixx="1" ixy="0" ixz="0"
-				 iyy="1" iyz="0" izz="1"/>
-		</inertial>
-		<visual name="base_visual">
-			<origin xyz="0 0 0" rpy="0 0 0"/>
-			<geometry name="pioneer_geom">
-				<mesh filename="package://p2os_urdf/meshes/p3dx_meshes/front_sonar.stl"/>
-			</geometry>
-			<material name="SonarYellow">
-				<color rgba="0.715 0.583 0.210 1.0"/>
-			</material>
-		</visual>
-		<collision>
-			<origin xyz="0 0 0" rpy="0 0 0"/>
-			<geometry>
-				<box size="0 0 0"/>
+		<parent link="caster_wheel"/>
+		<child link="caster_hubcap"/>
+	</joint>
+	<link name="left_hub">
+		<visual>
+			<origin xyz="0 0 0" rpy="0 0 0"/>
+			<geometry>
+				<mesh filename="package://amr_robots_description/meshes/p3dx_meshes/left_hubcap.stl"/>
+			</geometry>
+			<material name="HubcapYellow">
+				<color rgba="1.0 0.811 0.151 1.0"/>
+			</material>
+		</visual>
+		<collision>
+			<origin xyz="0 0 0" rpy="${-3.1415927/2.0} 0 0"/>
+			<geometry>
+				<!--<mesh filename="package://amr_robots_description/meshes/p3dx_meshes/caster_wheel.stl"/>-->
+				<cylinder radius="0.09" length="0.01"/>
 			</geometry>
 		</collision>
 	</link>
-	<joint name="base_front_joint" type="fixed">
-		<origin xyz="-0.198 0 0.208" rpy="0 0 0"/>
-		<parent link="base_link"/>
-		<child link="front_sonar"/>
-	</joint>
-	<joint name="base_back_joint" type="fixed">
-		<origin xyz="0.109 0 0.209" rpy="0 0 0"/>
-		<parent link="base_link"/>
-		<child link="back_sonar"/>
-	</joint>
-	<link name="back_sonar">
-		<inertial>
-			<mass value="0"/>
-			<origin xyz="0 0 0"/>
-			<inertia ixx="1" ixy="0" ixz="0"
-				 iyy="1" iyz="0" izz="1"/>
-		</inertial>
-		<visual name="base_visual">
-			<origin xyz="0 0 0" rpy="0 0 0"/>
-			<geometry name="pioneer_geom">
-				<mesh filename="package://p2os_urdf/meshes/p3dx_meshes/back_sonar.stl"/>
-			</geometry>
-			<material name="SonarYellow">
-				<color rgba="0.715 0.583 0.210 1.0"/>
-			</material>
-		</visual>
-		<collision>
-			<origin xyz="0 0 0" rpy="0 0 0"/>
-			<geometry>
-				<box size="0 0 0"/>
-			</geometry>
-		</collision>
-	</link>
+	<joint name="left_hub_joint" type="fixed">
+		<origin xyz="0 0.15 0.08" rpy="0 0 0"/>
+		<parent link="base_link"/>
+		<child link="left_hub"/>
+		<axis xyz="0 1 0"/>
+	</joint>
+	<link name="left_wheel_joint">
+		<visual>
+			<origin xyz="0 0 0" rpy="0 0 0"/>
+			<geometry>
+				<mesh filename="package://amr_robots_description/meshes/p3dx_meshes/left_wheel.stl"/>
+			</geometry>
+			<material name="WheelBlack">
+				<color rgba="0.117 0.117 0.117 1"/>
+			</material>
+		</visual>
+	</link>
+	<joint name="left_wheel_joint" type="fixed">
+		<origin xyz="0 0 0" rpy="0 0 0"/>
+		<parent link="left_hub"/>
+		<child link="left_wheel_joint"/>
+	</joint>
+	<gazebo reference="left_wheel_joint">
+		<material value="Gazebo/Black"/>
+	</gazebo>
+	<link name="right_hub">
+		<visual>
+			<origin xyz="0 0 0" rpy="0 0 0"/>
+			<geometry>
+				<mesh filename="package://amr_robots_description/meshes/p3dx_meshes/right_hubcap.stl"/>
+			</geometry>
+			<material name="HubcapYellow">
+				<color rgba="1.0 0.811 0.151 1.0"/>
+			</material>
+		</visual>
+		<collision>
+		<origin xyz="0 0 0" rpy="${-3.1415927/2.0} 0 0"/>
+		<geometry>
+			<!--<mesh filename="package://amr_robots_description/meshes/p3dx_meshes/caster_wheel.stl"/>-->
+			<cylinder radius="0.09" length="0.01"/>
+		</geometry>
+	</collision>
+	</link>
+	<gazebo reference="right_hub">
+		<material value="Gazebo/Yellow"/>
+	</gazebo>
+	<joint name="right_hub_joint" type="fixed">
+		<origin xyz="0 -0.15 0.08" rpy="0 0 0"/>
+		<parent link="base_link"/>
+		<child link="right_hub"/>
+		<axis xyz="0 1 0"/>
+	</joint>
+	<link name="right_wheel_joint">
+		<visual>
+			<origin xyz="0 0 0" rpy="0 0 0"/>
+			<geometry>
+				<mesh filename="package://amr_robots_description/meshes/p3dx_meshes/right_wheel.stl"/>
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
File: description/urdf/pioneer3dx_wheel.xacro (robot description, xacro)
@@ -6,9 +6,9 @@
   xmlns:xacro="http://ros.org/wiki/xacro"
   >
-  <!--<include filename="$(find p2os_urdf)/defs/materials.xacro"/>-->
+  <!--<include filename="$(find amr_robots_description)/urdf/materials.xacro"/>-->
   <!-- Properties (Constants) -->
   <property name="M_PI" value="3.14159"/>
 <!-- Right/Left Hubcap + Wheel -->
-<xacro:macro name="p3dx_wheel" params="suffix parent reflect">
+<xacro:macro name="p3dx_wheel" params="suffix reflect">
   <link name="p3dx_${suffix}_wheel">
     <inertial>
@@ -21,5 +21,5 @@
       <origin xyz="0 0 0" rpy="0 0 0"/>
       <geometry name="pioneer_geom">
-        <mesh filename="package://p2os_urdf/meshes/p3dx_meshes/${suffix}_wheel.stl"/>
+        <mesh filename="package://amr_robots_description/meshes/p3dx_meshes/${suffix}_wheel.stl"/>
       </geometry>
       <material name="WheelBlack">
@@ -30,5 +30,5 @@
       <origin xyz="0 0 0" rpy="${-3.1415927/2} 0 0"/>
       <geometry>
-        <!--<mesh filename="package://p2os_urdf/meshes/p3dx_meshes/${suffix}_wheel.stl"/>-->
+        <!--<mesh filename="package://amr_robots_description/meshes/p3dx_meshes/${suffix}_wheel.stl"/>-->
         <cylinder radius="0.09" length="0.01"/>
       </geometry>
@@ -51,5 +51,5 @@
     <origin xyz="0 0 0" rpy="0 0 0"/>
     <geometry name="pioneer_geom">
-      <mesh filename="package://p2os_urdf/meshes/p3dx_meshes/${suffix}_hubcap.stl"/>
+      <mesh filename="package://amr_robots_description/meshes/p3dx_meshes/${suffix}_hubcap.stl"/>
     </geometry>
     <material name="HubcapYellow">
@@ -64,5 +64,5 @@
   </collision>
   </link>
-  <transmission type="pr2_mechanism_model/SimpleTransmission" name="${parent}_${suffix}_wheel_trans">
+  <transmission type="pr2_mechanism_model/SimpleTransmission" name="${suffix}_wheel_trans">
     <actuator name="base_${suffix}_wheel_motor" />
     <joint name="base_${suffix}_wheel_joint" />
@@ -75,5 +75,5 @@
     <joint_properties damping="0.0" friction="0.0" />
     <origin xyz="0 ${reflect*0.158} 0.091" rpy="0 0 0"/>
-    <parent link="base_link"/>
+    <parent link="p3dx_${suffix}_hubcap"/>
     <child link="p3dx_${suffix}_wheel"/>
   </joint>

Commit message: Modified p3at macros, some gazebo-related stuff, annd more robust makefile

File: description/urdf/pioneer3at.urdf.xacro (robot description, xacro)
@@ -129,7 +129,7 @@
 		<child link="back_sonar"/>
 	</joint>
-<!-- Front Axles + Wheels + Hubcaps -->
-<xacro:macro name="p3at_front" params="suffix reflect">
-	<link name="p3at_front_${suffix}_axle">
+<xacro:macro name="p3at_drive_side" params="side reflect">
+  <!-- Front Axles + Wheels + Hubcaps -->
+	<link name="p3at_front_${side}_axle">
 		<inertial>
 			<mass value="0.1"/>
@@ -154,13 +154,13 @@
 	</collision>
 	</link>
-	<gazebo reference="p3at_front_${suffix}_axle">
+	<gazebo reference="p3at_front_${side}_axle">
 		<material value="Gazebo/Grey"/>
 	</gazebo>
-	<joint name="base_front_${suffix}_axle_joint" type="fixed">
+	<joint name="base_front_${side}_axle_joint" type="fixed">
 		<origin xyz="0.135 ${reflect*0.156} 0.111" rpy="0 0 0"/>
 		<parent link="base_link"/>
-		<child link="p3at_front_${suffix}_axle"/>
-	</joint>
-	<link name="p3at_front_${suffix}_hub">
+		<child link="p3at_front_${side}_axle"/>
+	</joint>
+	<link name="p3at_front_${side}_hub">
 		<inertial>
 			<mass value="0.1"/>
@@ -172,5 +172,5 @@
 		<origin xyz="0 0 0" rpy="0 0 0"/>
 		<geometry name="pioneer_geom">
-			<mesh filename="package://amr_robots_description/meshes/p3at_meshes/${suffix}_hubcap.stl"/>
+			<mesh filename="package://amr_robots_description/meshes/p3at_meshes/${side}_hubcap.stl"/>
 		</geometry>
 		<material name="HubcapYellow">
@@ -185,13 +185,13 @@
 	</collision>
 	</link>
-	<gazebo reference="p3at_front_${suffix}_hub">
+	<gazebo reference="p3at_front_${side}_hub">
 		<material value="Gazebo/Yellow"/>
 	</gazebo>
-	<joint name="base_front_${suffix}_hub_joint" type="fixed">
+	<joint name="base_front_${side}_hub_joint" type="fixed">
 		<origin xyz="0 ${reflect*0.041} 0" rpy="0 0 0"/>
-		<parent link="p3at_front_${suffix}_axle"/>
-		<child link="p3at_front_${suffix}_hub"/>
-	</joint>
-	<link name="p3at_front_${suffix}_wheel">
+		<parent link="p3at_front_${side}_axle"/>
+		<child link="p3at_front_${side}_hub"/>
+	</joint>
+	<link name="p3at_front_${side}_wheel">
 		<inertial>
 			<mass value="0.5"/>
@@ -217,8 +217,8 @@
 	</collision>
 	</link>
-	<gazebo reference="p3at_front_${suffix}_wheel">
+	<gazebo reference="p3at_front_${side}_wheel">
 		<material value="Gazebo/Black"/>
 	</gazebo>
-	<joint name="p3at_front_${suffix}_wheel_joint" type="continuous">
+	<joint name="p3at_front_${side}_wheel_joint" type="continuous">
   	<axis xyz="0 1 0"/>
     <anchor xyz="0 0 0"/>
@@ -226,9 +226,9 @@
     <joint_properties damping="0.7"/>
 		<origin xyz="0 0 0" rpy="0 0 0"/>
-		<parent link="p3at_front_${suffix}_hub"/>
-		<child link="p3at_front_${suffix}_wheel"/>
+		<parent link="p3at_front_${side}_hub"/>
+		<child link="p3at_front_${side}_wheel"/>
 	</joint>
 <!-- Back Axles + Wheels + Hubcaps -->
-	<link name="p3at_back_${suffix}_axle">
+	<link name="p3at_back_${side}_axle">
 		<inertial>
 			<mass value="0.1"/>
@@ -253,13 +253,13 @@
 	</collision>
 	</link>
-	<gazebo reference="p3at_back_${suffix}_axle">
+	<gazebo reference="p3at_back_${side}_axle">
 		<material value="Gazebo/Grey"/>
 	</gazebo>
-	<joint name="bp3at_back_${suffix}_axle_joint" type="fixed">
+	<joint name="bp3at_back_${side}_axle_joint" type="fixed">
 		<origin xyz="-0.134 ${reflect*0.156} 0.111" rpy="0 0 0"/>
 		<parent link="base_link"/>
-		<child link="p3at_back_${suffix}_axle"/>
-	</joint>
-	<link name="p3at_back_${suffix}_hub">
+		<child link="p3at_back_${side}_axle"/>
+	</joint>
+	<link name="p3at_back_${side}_hub">
 		<inertial>
 			<mass value="0.1"/>
@@ -271,5 +271,5 @@
 		<origin xyz="0 0 0" rpy="0 0 0"/>
 		<geometry name="pioneer_geom">
-			<mesh filename="package://amr_robots_description/meshes/p3at_meshes/${suffix}_hubcap.stl"/>
+			<mesh filename="package://amr_robots_description/meshes/p3at_meshes/${side}_hubcap.stl"/>
 		</geometry>
 		<material name="HubcapYellow"/>
@@ -278,17 +278,17 @@
 		<origin xyz="0 0 0" rpy="0 0 0"/>
 		<geometry>
-			<mesh filename="package://amr_robots_description/meshes/p3at_meshes/${suffix}_hubcap.stl"/>
-		</geometry>
-	</collision>
-	</link>
-	<gazebo reference="p3at_back_${suffix}_hub">
+			<mesh filename="package://amr_robots_description/meshes/p3at_meshes/${side}_hubcap.stl"/>
+		</geometry>
+	</collision>
+	</link>
+	<gazebo reference="p3at_back_${side}_hub">
 		<material value="Gazebo/Yellow"/>
 	</gazebo>
-	<joint name="p3at_back_${suffix}_hub_joint" type="fixed">
+	<joint name="p3at_back_${side}_hub_joint" type="fixed">
 		<origin xyz="-0 ${reflect*0.041} 0" rpy="0 0 0"/>
-		<parent link="p3at_back_${suffix}_axle"/>
-		<child link="p3at_back_${suffix}_hub"/>
-	</joint>
-	<link name="p3at_back_${suffix}_wheel">
+		<parent link="p3at_back_${side}_axle"/>
+		<child link="p3at_back_${side}_hub"/>
+	</joint>
+	<link name="p3at_back_${side}_wheel">
 		<inertial>
 			<mass value="0.5"/>
@@ -312,8 +312,8 @@
 	</collision>
 	</link>
-	<gazebo reference="p3at_back_${suffix}_wheel">
+	<gazebo reference="p3at_back_${side}_wheel">
 		<material value="Gazebo/Black"/>
 	</gazebo>
-	<joint name="p3at_back_${suffix}_wheel_joint" type="continuous">
+	<joint name="p3at_back_${side}_wheel_joint" type="continuous">
 	  <axis xyz="0 1 0"/>
     <anchor xyz="0 0 0"/>
@@ -321,8 +321,8 @@
     <joint_properties damping="0.7"/>
 		<origin xyz="0 0 0" rpy="0 0 0"/>
-		<parent link="p3at_back_${suffix}_hub"/>
-		<child link="p3at_back_${suffix}_wheel"/>
-	</joint>
-  <gazebo reference="p3at_back_${suffix}_wheel">
+		<parent link="p3at_back_${side}_hub"/>
+		<child link="p3at_back_${side}_wheel"/>
+	</joint>
+  <gazebo reference="p3at_back_${side}_wheel">
     <kp>1000000.0</kp> <!-- kp and kd for rubber -->
     <kd>100.0</kd>
@@ -333,5 +333,5 @@
     <minDepth>0.00</minDepth>
   </gazebo>
-  <gazebo reference="p3at_front_${suffix}_wheel">
+  <gazebo reference="p3at_front_${side}_wheel">
     <kp>1000000.0</kp> <!-- kp and kd for rubber -->
     <kd>100.0</kd>
@@ -360,8 +360,6 @@
 </gazebo>
 </xacro:macro>
-<xacro:p3at_front suffix="left" reflect="1"/>
-<xacro:p3at_front suffix="right" reflect="-1"/>
-<xacro:p3at_back suffix="left" reflect="1"/>
-<xacro:p3at_back suffix="right" reflect="-1"/>
+<xacro:p3at_drive_side side="left" reflect="1"/>
+<xacro:p3at_drive_side side="right" reflect="-1"/>
 <xacro:p3at_gazebo_ext/>
 </robot>

Commit message: minor updates to p3at gazebo properties, more helpful check for check_urdf in makefile

File: description/urdf/pioneer3at.urdf.xacro (robot description, xacro)
@@ -332,4 +332,5 @@
     <maxVel>1.0</maxVel>
     <minDepth>0.00</minDepth>
+    <material value="Gazebo/Black" />
   </gazebo>
   <gazebo reference="p3at_front_${side}_wheel">
@@ -341,4 +342,5 @@
     <maxVel>1.0</maxVel>
     <minDepth>0.00</minDepth>
+    <material value="Gazebo/Black" />
   </gazebo>
 </xacro:macro>
@@ -356,5 +358,8 @@
     <robotBaseFrame>base_link</robotBaseFrame>
     <torque>200</torque>
-    <topicName>cmd_vel</topicName>
+    <commandTopic>cmd_vel</commandTopic>
+    <odometryTopic>odom</odometryTopic>
+    <odometryFrame>odom</odometryFrame>
+    <broadcastTF>1</broadcastTF>
   </plugin>
 </gazebo>
