Commit message: added link for ekf

File: description/urdf/pioneer3at.urdf.xacro (robot description, xacro)
@@ -58,4 +58,18 @@
     <child link="imu_link"/>
   </joint>
+  <joint name="basefootprint_joint" type="fixed">
+    <axis xyz="1 0 0"/> <!-- 0 1 0 -->
+    <origin xyz="0 0 0.19"/>
+    <parent link="base_link"/>
+    <child link="base_footprint"/>
+  </joint>
+<link name="base_footprint">
+  <visual>
+    <origin rpy="0 0 0" xyz="0 0 0"/>
+    <geometry>
+      <box size="0.001 0.001 0.001"/>
+    </geometry>
+  </visual>
+</link>
 <link name="imu_link">
   <inertial>
@@ -406,5 +420,5 @@
         <topicName>imu_data</topicName>
         <serviceName>imu_service</serviceName>
-        <gaussianNoise>0.0</gaussianNoise>
+        <gaussianNoise>10.0</gaussianNoise>
         <updateRate>30.0</updateRate>
     </plugin>
@@ -430,4 +444,5 @@
     <bodyName>base_link</bodyName>
     <topicName>odom_gt</topicName>
+    <gaussianNoise>3.0</gaussianNoise>
     <updateRate>30.0</updateRate>
   </plugin>

Commit message: fixed colours

File: description/urdf/pioneer3at.urdf.xacro (robot description, xacro)
@@ -5,31 +5,6 @@
        xmlns:xacro="http://ros.org/wiki/xacro"
 name="pioneer3at">
-<xacro:include filename="$(find amr_robots_description)/urdf/materials.xacro" />
-<!-- Chassis -->
-	<link name="base_link">
-		<!--  For pointers on inertial and gazebo-related parameters see
-		       * http://wiki.ros.org/urdf/Tutorials/Adding%20Physical%20and%20Collision%20Properties%20to%20a%20URDF%20Model
-                       * http://answers.gazebosim.org/question/4372/the-inertia-matrix-explained/
-		       * http://gazebosim.org/tutorials?tut=inertia&cat=build_robot, and
-                       * http://gazebosim.org/tutorials/?tut=ros_urdf
-                       * http://en.wikipedia.org/wiki/List_of_moment_of_inertia_tensors
-                -->
-		<inertial>
-			<mass value="21.5"/> <!-- P3AT 18.6kg plus three batteries @ 2.4kg each  minus four wheels @ 1.4 kg ea and top plate @ 0.1 kg-->
-			<origin xyz="0 -0.1 0.177"/>
-			<inertia ixx="0.3338" ixy="0.0"     ixz="0.0"
-				              iyy="0.4783"  iyz="0.0"
-				                            izz="0.3338"/>
-		</inertial>
-		<visual name="base_visual">
-			<origin xyz="0 0 0.177" rpy="0 0 0"/>
-			<geometry name="pioneer_geom">
-				<mesh filename="package://amr_robots_description/meshes/p3at_meshes/chassis.stl"/>
-			</geometry>
-			<material name="ChassisRed">
-				<color rgba="0.851 0.0 0.0 1.0"/>
-			</material>
-		</visual>
-		<collision>
+    <link name="base_link">
+ <collision>
 			<origin xyz="0 0 0.177" rpy="0 0 0"/>
 				<geometry>
@@ -37,19 +12,19 @@
 				</geometry>
 		</collision>
-	</link>
-	<gazebo reference="base_link">
-      <material>
-         <!--
-      <script>
-         <uri>/usr/share/gazebo-7/media/materials/scripts/gazebo.material</uri>
-          <name>Gazebo/Green</name>
-      </script>
--->
-          <ambient>1 0 0 0</ambient>
-          <diffuse>1 0 0 0</diffuse>
-          <specular>0 0 0 1</specular>
-          <emissive>0 0 0 1</emissive>
-</material>
-	</gazebo>
+    <visual>
+    <origin xyz="0 0 0.177" rpy="0 0 0"/>
+	<geometry>
+        <mesh filename="package://amr_robots_description/meshes/p3at_meshes/chassis.stl"/>
+      </geometry>
+    </visual>
+<inertial>
+			<mass value="21.5"/> <!-- P3AT 18.6kg plus three batteries @ 2.4kg each  minus four wheels @ 1.4 kg ea and top plate @ 0.1 kg-->
+			<origin xyz="0 -0.1 0.177"/>
+			<inertia ixx="0.3338" ixy="0.0" ixz="0.0" iyy="0.4783" iyz="0.0" izz="0.3338"/>
+</inertial>
+  </link>
+  <gazebo reference="base_link">
+<material>Gazebo/Orange</material>
+  </gazebo>
   <joint name="imu_joint" type="fixed">
     <axis xyz="1 0 0"/> <!-- 0 1 0 -->
@@ -73,9 +48,10 @@
 </link>
 <link name="imu_link">
-  <inertial>
-    <mass value="0.001"/>
+   <collision>
     <origin rpy="0 0 0" xyz="0 0 0"/>
-    <inertia ixx="0.0001" ixy="0" ixz="0" iyy="0.000001" iyz="0" izz="0.0001"/>
-  </inertial>
+    <geometry>
+      <box size=".001 .001 .001"/>
+    </geometry>
+  </collision>
   <visual>
     <origin rpy="0 0 0" xyz="0 0 0"/>
@@ -84,71 +60,39 @@
     </geometry>
   </visual>
-  <collision>
+   <inertial>
+    <mass value="0.001"/>
     <origin rpy="0 0 0" xyz="0 0 0"/>
-    <geometry>
-      <box size=".001 .001 .001"/>
-    </geometry>
-  </collision>
+    <inertia ixx="0.0001" ixy="0" ixz="0" iyy="0.000001" iyz="0" izz="0.0001"/>
+  </inertial>
 </link>
 <!-- Top -->
-	<link name="top_plate">
-		<inertial>
-			<mass value="0.1"/>
-			<origin xyz="-0.025 0 -0.223"/>
-			<inertia ixx="1.0" ixy="0.0" ixz="0.0"
-				 iyy="1.0" iyz="0.0"
- 				izz="1.0"/>
-		</inertial>
-		<visual name="base_visual">
-			<origin xyz="0 0 0" rpy="0 0 0"/>
-			<geometry name="pioneer_geom">
-				<mesh filename="package://amr_robots_description/meshes/p3at_meshes/top.stl"/>
-			</geometry>
-			<material name="TopBlack">
-					<color rgba="0.038 0.038 0.038 1.0"/>
-			</material>
-		</visual>
-		<collision>
-			<origin xyz="0 0 0" rpy="0 0 0"/>
-			<geometry>
-				<box size="0.1 0.1 0.1"/>
-			</geometry>
-		</collision>
-	</link>
-	<gazebo reference="top_plate">
-    <material>Gazebo/Black</material>
-	</gazebo>
-	<joint name="base_top_joint" type="fixed">
+    <joint name="base_top_joint" type="fixed">
 		<origin xyz="0.003 0 0.274" rpy="0 0 0"/>
 		<parent link="base_link"/>
 		<child link="top_plate"/>
 	</joint>
+	<link name="top_plate">
+		<collision>
+			<origin xyz="0 0 0" rpy="0 0 0"/>
+			<geometry>
+				<box size="0.1 0.1 0.1"/>
+			</geometry>
+		</collision>
+		<visual>
+			<origin xyz="0 0 0" rpy="0 0 0"/>
+			<geometry>
+				<mesh filename="package://amr_robots_description/meshes/p3at_meshes/top.stl"/>
+			</geometry>
+		</visual>
+		<inertial>
+			<mass value="0.1"/>
+			<origin xyz="-0.025 0 -0.223"/>
+			<inertia ixx="1.0" ixy="0.0" ixz="0.0" iyy="1.0" iyz="0.0" izz="1.0"/>
+		</inertial>
+	</link>
+	<gazebo reference="top_plate">
+    <material>Gazebo/Blue</material>
+	</gazebo>
 <!-- Front + Back Sonar -->
-	<link name="front_sonar">
-		<inertial>
-			<mass value="0.1"/>
-			<origin xyz="0 0 0"/>
-			<inertia ixx="1.0" ixy="0.0" ixz="0.0"
-				 iyy="1.0" iyz="0.0" izz="1.0"/>
-		</inertial>
-		<visual name="base_visual">
-			<origin xyz="0 0 0" rpy="0 0 0"/>
-			<geometry name="pioneer_geom">
-				<mesh filename="package://amr_robots_description/meshes/p3at_meshes/front_sonar.stl"/>
-			</geometry>
-			<material name="SonarYellow">
-				<color rgba="0.715 0.583 0.210 1.0"/>
-			</material>
-		</visual>
-		<collision>
-			<origin xyz="0 0 0" rpy="0 0 0"/>
-			<geometry>
-				<box size="0.1 0.1 0.1"/>
-			</geometry>
-		</collision>
-	</link>
-	<gazebo reference="front_sonar">
-		<material value="Gazebo/Yellow"/>
-	</gazebo>
 	<joint name="base_front_joint" type="fixed">
 		<origin xyz="0.193 0 0.25" rpy="0 0 0"/>
@@ -156,38 +100,84 @@
 		<child link="front_sonar"/>
 	</joint>
-	<link name="back_sonar">
-		<inertial>
-			<mass value="0.1"/>
-			<origin xyz="0 0 0"/>
-			<inertia ixx="1.0" ixy="0.0" ixz="0.0"
-				 iyy="1.0" iyz="0.0" izz="1.0"/>
+	<link name="front_sonar">
+		<collision>
+			<origin xyz="0 0 0" rpy="0 0 0"/>
+			<geometry>
+				<box size="0.1 0.1 0.1"/>
+			</geometry>
+		</collision>
+		<visual>
+			<origin xyz="0 0 0" rpy="0 0 0"/>
+			<geometry>
+				<mesh filename="package://amr_robots_description/meshes/p3at_meshes/front_sonar.stl"/>
+			</geometry>
+		</visual>
+		<inertial>
+			<mass value="0.1"/>
+			<origin xyz="0 0 0"/>
+			<inertia ixx="1.0" ixy="0.0" ixz="0.0" iyy="1.0" iyz="0.0" izz="1.0"/>
 		</inertial>
-		<visual name="base_visual">
-			<origin xyz="0 0 0" rpy="0 0 0"/>
-			<geometry name="pioneer_geom">
-				<mesh filename="package://amr_robots_description/meshes/p3at_meshes/back_sonar.stl"/>
-			</geometry>
-			<material name="SonarYellow">
-				<color rgba="0.715 0.583 0.210 1.0"/>
-			</material>
-		</visual>
-		<collision>
-			<origin xyz="0 0 0" rpy="0 0 0"/>
-			<geometry>
-				<box size="0.1 0.1 0.1"/>
-			</geometry>
-		</collision>
-	</link>
-	<gazebo reference="back_sonar">
-		<material value="Gazebo/Yellow"/>
-	</gazebo>
-	<joint name="base_back_joint" type="fixed">
+	</link>
+    <gazebo reference="front_sonar">
+    <material>Gazebo/Yellow</material>
+	</gazebo>
+   <joint name="base_back_joint" type="fixed">
 		<origin xyz="-0.187 0 0.247" rpy="0 0 0"/>
 		<parent link="base_link"/>
 		<child link="back_sonar"/>
 	</joint>
+    <link name="back_sonar">
+		<collision>
+			<origin xyz="0 0 0" rpy="0 0 0"/>
+			<geometry>
+				<box size="0.1 0.1 0.1"/>
+			</geometry>
+		</collision>
+		<visual>
+			<origin xyz="0 0 0" rpy="0 0 0"/>
+			<geometry>
+				<mesh filename="package://amr_robots_description/meshes/p3at_meshes/back_sonar.stl"/>
+			</geometry>
+		</visual>
+		<inertial>
+			<mass value="0.1"/>
+			<origin xyz="0 0 0"/>
+			<inertia ixx="1.0" ixy="0.0" ixz="0.0" iyy="1.0" iyz="0.0" izz="1.0"/>
+		</inertial>
+	</link>
+	<gazebo reference="back_sonar">
+		<material>Gazebo/Yellow</material>
+	</gazebo>
 <xacro:macro name="p3at_drive_side" params="side reflect">
   <!-- Front Axles + Wheels + Hubcaps -->
 	<link name="p3at_front_${side}_axle">
+		<inertial>
+			<mass value="0.1"/>
+			<origin xyz="0 0 0"/>
+			<inertia ixx="1.0" ixy="0.0" ixz="0.0"
+				 iyy="1.0" iyz="0.0" izz="1.0"/>
+  	 	</inertial>
+	<visual>
+		<origin xyz="0 0 0" rpy="0 0 0"/>
+		<geometry>
+			<mesh filename="package://amr_robots_description/meshes/p3at_meshes/axle.stl"/>
+		</geometry>
+	</visual>
+	<collision>
+		<origin xyz="0 0 0" rpy="0 0 0"/>
+		<geometry>
+			<box size="0.1 0.1 0.1"/>
+		</geometry>
+	</collision>
+	</link>
+	<gazebo reference="p3at_front_${side}_axle">
+		<material>Gazebo/Green</material>
+	</gazebo>
+	<joint name="base_front_${side}_axle_joint" type="fixed">
+		<origin xyz="0.135 ${reflect*0.156} 0.111" rpy="0 0 0"/>
+		<parent link="base_link"/>
+		<child link="p3at_front_${side}_axle"/>
+	</joint>
+	<link name="p3at_front_${side}_hub">
 		<inertial>
 			<mass value="0.1"/>
@@ -199,35 +189,4 @@
 		<origin xyz="0 0 0" rpy="0 0 0"/>
 		<geometry name="pioneer_geom">
-			<mesh filename="package://amr_robots_description/meshes/p3at_meshes/axle.stl"/>
-		</geometry>
-		<material name="AxleGrey">
-			<color rgba="0.5 0.5 0.5 1"/>
-		</material>
-	</visual>
-	<collision>
-		<origin xyz="0 0 0" rpy="0 0 0"/>
-		<geometry>
-			<box size="0.1 0.1 0.1"/>
-		</geometry>
-	</collision>
-	</link>
-	<gazebo reference="p3at_front_${side}_axle">
-		<material value="Gazebo/Grey"/>
-	</gazebo>
-	<joint name="base_front_${side}_axle_joint" type="fixed">
-		<origin xyz="0.135 ${reflect*0.156} 0.111" rpy="0 0 0"/>
-		<parent link="base_link"/>
-		<child link="p3at_front_${side}_axle"/>
-	</joint>
-	<link name="p3at_front_${side}_hub">
-		<inertial>
-			<mass value="0.1"/>
-			<origin xyz="0 0 0"/>
-			<inertia ixx="1.0" ixy="0.0" ixz="0.0"
-				 iyy="1.0" iyz="0.0" izz="1.0"/>
-  	 	</inertial>
-	<visual name="base_visual">
-		<origin xyz="0 0 0" rpy="0 0 0"/>
-		<geometry name="pioneer_geom">
 			<mesh filename="package://amr_robots_description/meshes/p3at_meshes/${side}_hubcap.stl"/>
 		</geometry>
@@ -258,7 +217,7 @@
          iyy="0.015218160428" iyz="0" izz="0.011763977943"/>
       </inertial>
-	<visual name="base_visual">
-		<origin xyz="0 0 0" rpy="0 0 0"/>
-		<geometry name="pioneer_geom">
+	<visual>
+		<origin xyz="0 0 0" rpy="0 0 0"/>
+		<geometry>
 			<mesh filename="package://amr_robots_description/meshes/p3at_meshes/wheel.stl"/>
 		</geometry>
@@ -276,5 +235,5 @@
 	</link>
 	<gazebo reference="p3at_front_${side}_wheel">
-		<material value="Gazebo/Black"/>
+		<material>Gazebo/Black</material>
 	</gazebo>
 	<joint name="p3at_front_${side}_wheel_joint" type="continuous">
@@ -295,7 +254,7 @@
 				 iyy="1.0" iyz="0.0" izz="1.0"/>
   	 	</inertial>
-	<visual name="base_visual">
-		<origin xyz="0 0 0" rpy="0 0 0"/>
-		<geometry name="pioneer_geom">
+	<visual>
+		<origin xyz="0 0 0" rpy="0 0 0"/>
+		<geometry>
 			<mesh filename="package://amr_robots_description/meshes/p3at_meshes/axle.stl"/>
 		</geometry>
@@ -312,5 +271,5 @@
 	</link>
 	<gazebo reference="p3at_back_${side}_axle">
-		<material value="Gazebo/Grey"/>
+		<material value="Gazebo/Green"/>
 	</gazebo>
 	<joint name="p3at_back_${side}_axle_joint" type="fixed">
@@ -356,10 +315,9 @@
                                                                            izz="0.011763977943"/>
       </inertial>
-	<visual name="base_visual">
-		<origin xyz="0 0 0" rpy="0 0 0"/>
-		<geometry name="pioneer_geom">
+	<visual>
+		<origin xyz="0 0 0" rpy="0 0 0"/>
+		<geometry>
 			<mesh filename="package://amr_robots_description/meshes/p3at_meshes/wheel.stl"/>
 		</geometry>
-		<material name="WheelBlack"/>
 	</visual>
 	<collision>
@@ -372,5 +330,5 @@
 	</link>
 	<gazebo reference="p3at_back_${side}_wheel">
-		<material value="Gazebo/Black"/>
+		<material>Gazebo/Black</material>
 	</gazebo>
 	<joint name="p3at_back_${side}_wheel_joint" type="continuous">

Commit message: Fix P3AT inertial origin (x and y swapped so it was on the right side of the robot rather than towards the back a bit)

File: description/urdf/pioneer3at.urdf.xacro (robot description, xacro)
@@ -16,5 +16,5 @@
 		<inertial>
 			<mass value="21.5"/> <!-- P3AT 18.6kg plus three batteries @ 2.4kg each  minus four wheels @ 1.4 kg ea and top plate @ 0.1 kg-->
-			<origin xyz="0 -0.1 0.177"/>
+			<origin xyz="-0.1 0 0.177"/>
 			<inertia ixx="0.3338" ixy="0.0"     ixz="0.0"
 				              iyy="0.4783"  iyz="0.0"
